File: Hartware_2.0.0/7SEGMENTOS_X_3.sch (KiCad schematic (older format))
At the start: 10 parts, among them Q1 2N3904, Q2 2N3904, Q3 2N3904, U8 HDC-5633

Commit message: primer trabajo de codificacion
Parts:
- removed U8: HDC-5633, LIB:7seg-HDC-19x37.5mm, symbol D21_2550-rescue:HDC-5633-RESCUE-D21_2550
- added D11: LTC-4724JR, Devices_MSS:LTC-4724JR, symbol Mss_devices:LTC-4724JR
- Q1, Q2, Q3: value 2N3904 -> FZT493TA; footprint TO_SOT_Packages_SMD:SOT-23_Handsoldering -> Package_TO_SOT_SMD:SOT-223; symbol D21_2550-rescue:Q_NPN_CBE-RESCUE-D21_2550 -> Device:Q_NPN_CBE; Campo4 (none) -> FZT493TA
- R12, R13, R14: footprint Resistors_SMD:R_0805_HandSoldering -> Resistor_SMD:R_0805_2012Metric_Pad1.15x1.50mm_HandSolder; symbol D21_2550-rescue:R-RESCUE-D21_2550 -> Device:R; Campo4 (none) -> ERA-6AEB272V
- R15, R16, R17: footprint Resistors_ThroughHole:Resistor_Horizontal_RM10mm -> Resistor_SMD:R_2512_6332Metric_Pad1.34x3.40mm_HandSolder; symbol D21_2550-rescue:R-RESCUE-D21_2550 -> Device:R; Campo4 (none) -> RC2512JK-0722RL
Connections:
- wire segments 72 -> 25
- no-connect marks 3 -> 1
