File: Hartware_2.0.0/FuenteST.sch (KiCad schematic (older format))
At the start: 9 parts

Commit message: primer trabajo de codificacion
Parts:
- C1: symbol D21_2550-rescue:CP1-RESCUE-D21_2550 -> Device:CP1
- C8: symbol D21_2550-rescue:C-RESCUE-D21_2550 -> Device:C
- D1, D2, D3, D4: symbol D21_2550-rescue:D-RESCUE-D21_2550 -> Device:D
- D5: symbol D21_2550-rescue:D_Zener-RESCUE-D21_2550 -> Device:D_Zener
- R1: symbol D21_2550-rescue:R-RESCUE-D21_2550 -> Device:R
- R27: footprint Resistors_SMD:R_0805_HandSoldering -> Resistor_SMD:R_0805_2012Metric_Pad1.15x1.50mm_HandSolder; symbol D21_2550-rescue:R-RESCUE-D21_2550 -> Device:R
Changed lines of the file:
@@
 Comment4 ""
 $EndDescr
-Text GLabel 1700 3200 0    60   Input ~ 0
+Text GLabel 3750 3600 0    60   Input ~ 0
 Nac
-Text GLabel 1700 3000 0    60   Input ~ 0
+Text GLabel 3750 3400 0    60   Input ~ 0
 Vac
 $Comp
-L D21_2550-rescue:D_Zener-RESCUE-D21_2550 D5
+L Device:D_Zener D5
 U 1 1 56F22E6D
-P 5350 2950
-F 0 "D5" H 5350 3050 50  0000 C CNN
-F 1 "1N4733A" H 5350 2850 50  0000 C CNN
-F 2 "Diodes_ThroughHole:Diode_DO-35_SOD27_Horizontal_RM10" H 5350 2950 50  0001 C CNN
-F 3 "" H 5350 2950 50  0000 C CNN
-	1    5350 2950
+P 7400 3350
+F 0 "D5" H 7400 3450 50  0000 C CNN
+F 1 "1N4733A" H 7400 3250 50  0000 C CNN
+F 2 "Diodes_ThroughHole:Diode_DO-35_SOD27_Horizontal_RM10" H 7400 3350 50  0001 C CNN
+F 3 "" H 7400 3350 50  0000 C CNN
+	1    7400 3350
 	0    1    1    0
 $EndComp
-Text GLabel 5350 2050 1    60   Input ~ 0
+Text GLabel 7400 2450 1    60   Input ~ 0
 VDD
 $Comp
-L D21_2550-rescue:CP1-RESCUE-D21_2550 C1
+L Device:CP1 C1
 U 1 1 56F69FA4
-P 4550 3000
-F 0 "C1" H 4600 3100 50  0000 L CNN
-F 1 "680uf" H 4600 2900 50  0000 L CNN
-F 2 "Capacitors_ThroughHole:C_Radial_D8_L11.5_P3.5" H 4550 3000 60  0001 C CNN
-F 3 "" H 4550 3000 60  0000 C CNN
-	1    4550 3000
+P 6600 3400
+F 0 "C1" H 6650 3500 50  0000 L CNN
+F 1 "680uf" H 6650 3300 50  0000 L CNN
+F 2 "Capacitors_ThroughHole:C_Radial_D8_L11.5_P3.5" H 6600 3400 60  0001 C CNN
+F 3 "" H 6600 3400 60  0000 C CNN
+	1    6600 3400
 	1    0    0    -1
 $EndComp
 $Comp
-L D21_2550-rescue:R-RESCUE-D21_2550 R1
+L Device:R R1
 U 1 1 56F82842
-P 2600 2750
-F 0 "R1" V 2680 2750 40  0000 C CNN
-F 1 "300k" V 2607 2751 40  0000 C CNN
-F 2 "Resistors_ThroughHole:Resistor_Horizontal_RM10mm" V 2530 2750 30  0001 C CNN
-F 3 "" H 2600 2750 30  0000 C CNN
-	1    2600 2750
+P 4650 3150
+F 0 "R1" V 4730 3150 40  0000 C CNN
+F 1 "300k" V 4657 3151 40  0000 C CNN
+F 2 "Resistors_ThroughHole:Resistor_Horizontal_RM10mm" V 4580 3150 30  0001 C CNN
+F 3 "" H 4650 3150 30  0000 C CNN
+	1    4650 3150
 	0    1    1    0
 $EndComp
 Wire Wire Line
-	3400 2200 3800 2200
+	5450 2600 5850 2600
 Wire Wire Line
-	3800 2200 4550 2200
+	5850 2600 6600 2600
 Wire Wire Line
-	4550 2200 4800 2200
+	6600 2600 6850 2600
 Wire Wire Line
-	3400 3950 3800 3950
+	5450 4350 5850 4350
 Wire Wire Line
-	3800 3950 4000 3950
+	5850 4350 6050 4350
 Wire Wire Line
-	4000 3950 4550 3950
+	6050 4350 6600 4350
 Wire Wire Line
-	4550 3950 5350 3950
-Connection ~ 3800 3200
-Connection ~ 3400 3000
-Connection ~ 3800 2200
-Connection ~ 3800 3950
-Connection ~ 4550 2200
+	6600 4350 7400 4350
+Connection ~ 5850 3600
+Connection ~ 5450 3400
+Connection ~ 5850 2600
+Connection ~ 5850 4350
+Connection ~ 6600 2600
 Wire Wire Line
-	4000 3950 4000 4050
-Connection ~ 4000 3950
+	6050 4350 6050 4450
+Connection ~ 6050 4350
 Wire Wire Line
-	3400 3950 3400 3650
+	5450 4350 5450 4050
 Wire Wire Line
-	3800 3650 3800 3950
+	5850 4050 5850 4350
 Wire Wire Line
-	3800 2750 3800 3200
+	5850 3150 5850 3600
 Wire Wire Line
-	3800 3200 3800 3350
+	5850 3600 5850 3750
 Wire Wire Line
-	3400 2750 3400 3000
+	5450 3150 5450 3400
 Wire Wire Line
-	3400 3000 3400 3350
+	5450 3400 5450 3750
 Wire Wire Line
-	3400 2450 3400 2200
+	5450 2850 5450 2600
 Wire Wire Line
-	3800 2450 3800 2200
+	5850 2850 5850 2600
 Wire Wire Line
-	4550 3150 4550 3950
+	6600 3550 6600 4350
 Wire Wire Line
-	1700 3200 3800 3200
+	3750 3600 5850 3600
 $Comp
-L D21_2550-rescue:D-RESCUE-D21_2550 D1
+L Device:D D1
 U 1 1 56FC9299
-P 3400 2600
-F 0 "D1" H 3400 2700 50  0000 C CNN
-F 1 "1N4007" H 3400 2500 50  0000 C CNN
-F 2 "Diodes_ThroughHole:Diode_DO-41_SOD81_Horizontal_RM10" H 3400 2600 50  0001 C CNN
-F 3 "" H 3400 2600 50  0000 C CNN
-	1    3400 2600
+P 5450 3000
+F 0 "D1" H 5450 3100 50  0000 C CNN
+F 1 "1N4007" H 5450 2900 50  0000 C CNN
+F 2 "Diodes_ThroughHole:Diode_DO-41_SOD81_Horizontal_RM10" H 5450 3000 50  0001 C CNN
+F 3 "" H 5450 3000 50  0000 C CNN
+	1    5450 3000
 	0    1    1    0
 $EndComp
 $Comp
-L D21_2550-rescue:D-RESCUE-D21_2550 D3
+L Device:D D3
 U 1 1 56FC930C
-P 3800 2600
-F 0 "D3" H 3800 2700 50  0000 C CNN
-F 1 "1N4007" H 3800 2500 50  0000 C CNN
-F 2 "Diodes_ThroughHole:Diode_DO-41_SOD81_Horizontal_RM10" H 3800 2600 50  0001 C CNN
-F 3 "" H 3800 2600 50  0000 C CNN
-	1    3800 2600
+P 5850 3000
+F 0 "D3" H 5850 3100 50  0000 C CNN
+F 1 "1N4007" H 5850 2900 50  0000 C CNN
+F 2 "Diodes_ThroughHole:Diode_DO-41_SOD81_Horizontal_RM10" H 5850 3000 50  0001 C CNN
+F 3 "" H 5850 3000 50  0000 C CNN
+	1    5850 3000
 	0    1    1    0
 $EndComp
 $Comp
-L D21_2550-rescue:D-RESCUE-D21_2550 D2
+L Device:D D2
 U 1 1 56FC93DD
-P 3400 3500
-F 0 "D2" H 3400 3600 50  0000 C CNN
-F 1 "1N4007" H 3400 3400 50  0000 C CNN
-F 2 "Diodes_ThroughHole:Diode_DO-41_SOD81_Horizontal_RM10" H 3400 3500 50  0001 C CNN
-F 3 "" H 3400 3500 50  0000 C CNN
-	1    3400 3500
+P 5450 3900
+F 0 "D2" H 5450 4000 50  0000 C CNN
+F 1 "1N4007" H 5450 3800 50  0000 C CNN
+F 2 "Diodes_ThroughHole:Diode_DO-41_SOD81_Horizontal_RM10" H 5450 3900 50  0001 C CNN
+F 3 "" H 5450 3900 50  0000 C CNN
+	1    5450 3900
 	0    1    1    0
 $EndComp
 $Comp
-L D21_2550-rescue:D-RESCUE-D21_2550 D4
+L Device:D D4
 U 1 1 56FC9402
-P 3800 3500
-F 0 "D4" H 3800 3600 50  0000 C CNN
-F 1 "1N4007" H 3800 3400 50  0000 C CNN
-F 2 "Diodes_ThroughHole:Diode_DO-41_SOD81_Horizontal_RM10" H 3800 3500 50  0001 C CNN
-F 3 "" H 3800 3500 50  0000 C CNN
-	1    3800 3500
+P 5850 3900
+F 0 "D4" H 5850 4000 50  0000 C CNN
+F 1 "1N4007" H 5850 3800 50  0000 C CNN
+F 2 "Diodes_ThroughHole:Diode_DO-41_SOD81_Horizontal_RM10" H 5850 3900 50  0001 C CNN
+F 3 "" H 5850 3900 50  0000 C CNN
+	1    5850 3900
 	0    1    1    0
 $EndComp
@@
 L power1:GND #PWR01
 U 1 1 56FDA682
-P 4000 4050
-F 0 "#PWR01" H 4000 3800 50  0001 C CNN
-F 1 "GND" H 4000 3900 50  0000 C CNN
-F 2 "" H 4000 4050 50  0000 C CNN
-F 3 "" H 4000 4050 50  0000 C CNN
-	1    4000 4050
+P 6050 4450
+F 0 "#PWR01" H 6050 4200 50  0001 C CNN
+F 1 "GND" H 6050 4300 50  0000 C CNN
+F 2 "" H 6050 4450 50  0000 C CNN
+F 3 "" H 6050 4450 50  0000 C CNN
+	1    6050 4450
 	1    0    0    -1
 $EndComp
 $Comp
-L D21_2550-rescue:C-RESCUE-D21_2550 C8
+L Device:C C8
 U 1 1 5702B30B
-P 2600 3000
+P 4650 3400
 AR Path="/5702B30B" Ref="C8"  Part="1"
 AR Path="/56D4C312/5702B30B" Ref="C8"  Part="1"
-F 0 "C8" H 2625 3100 50  0000 L CNN
-F 1 "4.7uf" H 2625 2900 50  0000 L CNN
-F 2 "Choke_Axial_ThroughHole:Choke_Horizontal_RM25mm" H 2638 2850 50  0001 C CNN
-F 3 "" H 2600 3000 50  0000 C CNN
-	1    2600 3000
+F 0 "C8" H 4675 3500 50  0000 L CNN
+F 1 "4.7uf" H 4675 3300 50  0000 L CNN
+F 2 "Choke_Axial_ThroughHole:Choke_Horizontal_RM25mm" H 4688 3250 50  0001 C CNN
+F 3 "" H 4650 3400 50  0000 C CNN
+	1    4650 3400
 	0    1    1    0
 $EndComp
 Wire Wire Line
-	2750 3000 3000 3000
+	4800 3400 5050 3400
 Wire Wire Line
-	3000 3000 3400 3000
+	5050 3400 5450 3400
 Wire Wire Line
-	2450 3000 2200 3000
+	4500 3400 4250 3400
 Wire Wire Line
-	2200 3000 1700 3000
+	4250 3400 3750 3400
 Wire Wire Line
-	2450 2750 2200 2750
+	4500 3150 4250 3150
 Wire Wire Line
-	2200 2750 2200 3000
-Connection ~ 2200 3000
+	4250 3150 4250 3400
+Connection ~ 4250 3400
 Wire Wire Line
-	2750 2750 3000 2750
+	4800 3150 5050 3150
 Wire Wire Line
-	3000 2750 3000 3000
-Connection ~ 3000 3000
+	5050 3150 5050 3400
+Connection ~ 5050 3400
 $Comp
-L D21_2550-rescue:R-RESCUE-D21_2550 R27
+L Device:R R27
 U 1 1 5702BA59
-P 4950 2200
-F 0 "R27" V 5030 2200 50  0000 C CNN
-F 1 "100" V 4950 2200 50  0000 C CNN
-F 2 "Resistors_SMD:R_0805_HandSoldering" V 4880 2200 50  0001 C CNN
-F 3 "" H 4950 2200 50  0000 C CNN
-	1    4950 2200
+P 7000 2600
+F 0 "R27" V 7080 2600 50  0000 C CNN
+F 1 "100" V 7000 2600 50  0000 C CNN
+F 2 "Resistor_SMD:R_0805_2012Metric_Pad1.15x1.50mm_HandSolder" V 6930 2600 50  0001 C CNN
+F 3 "" H 7000 2600 50  0000 C CNN
+	1    7000 2600
 	0    1    1    0
 $EndComp
 Wire Wire Line
-	5100 2200 5350 2200
+	7150 2600 7400 2600
 Wire Wire Line
-	5350 2050 5350 2200
+	7400 2450 7400 2600
 Wire Wire Line
-	5350 2200 5350 2800
-Connection ~ 5350 2200
+	7400 2600 7400 3200
+Connection ~ 7400 2600
 Wire Wire Line
-	4550 2850 4550 2200
+	6600 3250 6600 2600
 Wire Wire Line
-	5350 3950 5350 3100
-Connection ~ 4550 3950
+	7400 4350 7400 3500
+Connection ~ 6600 4350
 $EndSCHEMATC

Commit message: modificacion de cartas
Parts:
- removed D1, D2, D3, D4: 1N4007, Diodes_ThroughHole:Diode_DO-41_SOD81_Horizontal_RM10, symbol Device:D
- removed D5: 1N4733A, Diodes_ThroughHole:Diode_DO-35_SOD27_Horizontal_RM10, symbol Device:D_Zener
- removed R27: 100, Resistor_SMD:R_0805_2012Metric_Pad1.15x1.50mm_HandSolder, symbol Device:R
- added C10, C9: CP1, Capacitor_SMD:CP_Elec_3x5.3, symbol Device:CP1
- added C11: 4,7uF, Capacitor_THT:CP_Radial_D8.0mm_P3.50mm, symbol Device:CP1
- added L1: SDR0503-472JL, Devices_MSS:SDR0503-XXX, symbol Device:L_Core_Ferrite
- added L2: 74479776247, Inductor_SMD:L_0805_2012Metric_Pad1.15x1.50mm_HandSolder, symbol Device:L_Core_Ferrite
- added RV1: B72214S0351K101, Capacitor_THT:C_Disc_D4.3mm_W1.9mm_P5.00mm, symbol Device:Varistor
- added TH1: Thermistor_NTC, Resistor_SMD:R_0805_2012Metric_Pad1.15x1.50mm_HandSolder, symbol Device:Thermistor_NTC
- added U8: PBO-3-S5, Devices_MSS:PBO-3-S5, symbol Mss_devices:PBO-3-S5
- C1: value 680uf -> 4,7uF; footprint Capacitors_ThroughHole:C_Radial_D8_L11.5_P3.5 -> Capacitor_THT:CP_Radial_D8.0mm_P3.50mm; Campo4 (none) -> A759KS475M2EAAE496
- C8: value 4.7uf -> 1nF; footprint Choke_Axial_ThroughHole:Choke_Horizontal_RM25mm -> Capacitor_SMD:C_0805_2012Metric_Pad1.15x1.50mm_HandSolder; Campo4 (none) -> C2012C0G2W102J060AA
- R1: footprint Resistors_ThroughHole:Resistor_Horizontal_RM10mm -> Resistor_SMD:R_1206_3216Metric_Pad1.24x1.80mm_HandSolder
Connections:
- wire segments 31 -> 34

Commit message: a medio hacer
Parts:
- added C12: 100nF, Capacitor_SMD:C_1206_3216Metric_Pad1.24x1.80mm_HandSolder, symbol Device:C
- C10: value CP1 -> 68uF; footprint Capacitor_SMD:CP_Elec_3x5.3 -> Capacitor_SMD:CP_Elec_6.3x7.7; Campo4 (none) -> UUD1V680MCL1GS
- C9: value CP1 -> 270uF; footprint Capacitor_SMD:CP_Elec_3x5.3 -> Capacitor_SMD:CP_Elec_6.3x7.7; Campo4 (none) -> EEE-FKC271XSP
Connections:
- net labels added: VO
- wire segments 34 -> 38
Changed lines of the file:
@@
 Text GLabel 3650 3650 0    60   Input ~ 0
 Vac
-Text GLabel 8050 3650 2    60   Output ~ 0
+Text GLabel 8350 3650 2    60   Output ~ 0
 VDD
 $Comp
@@
 P 7250 3850
 F 0 "C9" H 7365 3896 50  0000 L CNN
-F 1 "CP1" H 7365 3805 50  0000 L CNN
-F 2 "Capacitor_SMD:CP_Elec_3x5.3" H 7250 3850 50  0001 C CNN
-F 3 "~" H 7250 3850 50  0001 C CNN
+F 1 "270uF" H 7365 3805 50  0000 L CNN
+F 2 "Capacitor_SMD:CP_Elec_6.3x7.7" H 7250 3850 50  0001 C CNN
+F 3 "https://media.digikey.com/pdf/Data%20Sheets/Panasonic%20Capacitors%20PDFs/FKS_Series_Type_V.pdf" H 7250 3850 50  0001 C CNN
+F 4 "EEE-FKC271XSP" H 7250 3850 50  0001 C CNN "Campo4"
 	1    7250 3850
 	1    0    0    -1
@@
 P 7750 3850
 F 0 "C10" H 7865 3896 50  0000 L CNN
-F 1 "CP1" H 7865 3805 50  0000 L CNN
-F 2 "Capacitor_SMD:CP_Elec_3x5.3" H 7750 3850 50  0001 C CNN
-F 3 "~" H 7750 3850 50  0001 C CNN
+F 1 "68uF" H 7865 3805 50  0000 L CNN
+F 2 "Capacitor_SMD:CP_Elec_6.3x7.7" H 7750 3850 50  0001 C CNN
+F 3 "http://nichicon-us.com/english/products/pdfs/e-uud.pdf" H 7750 3850 50  0001 C CNN
+F 4 "UUD1V680MCL1GS" H 7750 3850 50  0001 C CNN "Campo4"
 	1    7750 3850
 	1    0    0    -1
@@
 Wire Wire Line
 	7250 4350 7250 4050
-Wire Wire Line
-	8050 3650 7750 3650
 Connection ~ 7750 3650
 $Comp
@@
 Wire Wire Line
 	4900 4100 4900 4050
+Text Label 7100 3650 0    60   ~ 0
+VO
+$Comp
+L Device:C C12
+U 1 1 5A7F66F8
+P 8200 3850
+F 0 "C12" H 8315 3896 50  0000 L CNN
+F 1 "100nF" H 8315 3805 50  0000 L CNN
+F 2 "Capacitor_SMD:C_1206_3216Metric_Pad1.24x1.80mm_HandSolder" H 8238 3700 50  0001 C CNN
+F 3 "https://search.kemet.com/component-edge/download/datasheet/C1206C104K5RACTU.pdf" H 8200 3850 50  0001 C CNN
+F 4 "C1206C104K5RAC7867" H 8200 3850 50  0001 C CNN "Campo4"
+	1    8200 3850
+	1    0    0    -1
+$EndComp
+Wire Wire Line
+	8200 3700 8200 3650
+Wire Wire Line
+	7750 3650 8200 3650
+Wire Wire Line
+	8350 3650 8200 3650
+Connection ~ 8200 3650
+Wire Wire Line
+	8200 4000 8200 4050
+Wire Wire Line
+	8200 4050 7750 4050
 $EndSCHEMATC

Commit message: finalinzando la placa
Parts:
- removed TH1: Thermistor_NTC, Resistor_SMD:R_0805_2012Metric_Pad1.15x1.50mm_HandSolder, symbol Device:Thermistor_NTC
Connections:
- wire segments 38 -> 37
Changed lines of the file:
@@
 L Device:R R1
 U 1 1 56F82842
-P 4900 3650
-F 0 "R1" V 4980 3650 40  0000 C CNN
-F 1 "300k" V 4907 3651 40  0000 C CNN
-F 2 "Resistor_SMD:R_1206_3216Metric_Pad1.24x1.80mm_HandSolder" V 4830 3650 30  0001 C CNN
-F 3 "" H 4900 3650 30  0000 C CNN
-	1    4900 3650
+P 4600 3650
+F 0 "R1" V 4680 3650 40  0000 C CNN
+F 1 "300k" V 4607 3651 40  0000 C CNN
+F 2 "Resistor_SMD:R_1206_3216Metric_Pad1.24x1.80mm_HandSolder" V 4530 3650 30  0001 C CNN
+F 3 "" H 4600 3650 30  0000 C CNN
+	1    4600 3650
 	0    1    1    0
 $EndComp
@@
 	5850 3750 5200 3750
 Wire Wire Line
-	5850 3950 5400 3950
-Wire Wire Line
-	5400 3950 5400 4100
-Wire Wire Line
-	5400 4100 5200 4100
+	5850 3950 5700 3950
+Wire Wire Line
+	5700 3950 5700 4100
+Wire Wire Line
+	5700 4100 5200 4100
 Wire Wire Line
 	5200 4100 5200 4050
 Wire Wire Line
-	5850 4050 5550 4050
-Wire Wire Line
-	5550 4050 5550 4250
-Wire Wire Line
-	5550 4250 4200 4250
+	5850 4050 5750 4050
+Wire Wire Line
+	5750 4050 5750 4250
+Wire Wire Line
+	5750 4250 4200 4250
 $Comp
 L Device:L_Core_Ferrite L1
@@
 	5550 3650 5850 3650
 Wire Wire Line
-	5250 3650 5050 3650
-$Comp
-L Device:Thermistor_NTC TH1
-U 1 1 5A7D09D6
-P 4450 3650
-F 0 "TH1" V 4160 3650 50  0000 C CNN
-F 1 "Thermistor_NTC" V 4251 3650 50  0000 C CNN
-F 2 "Resistor_SMD:R_0805_2012Metric_Pad1.15x1.50mm_HandSolder" H 4450 3700 50  0001 C CNN
-F 3 "~" H 4450 3700 50  0001 C CNN
-	1    4450 3650
-	0    1    1    0
-$EndComp
-Wire Wire Line
-	4600 3650 4750 3650
+	5250 3650 4750 3650
 $Comp
 L Device:Varistor RV1
@@
 Wire Wire Line
 	4200 3800 4200 3650
-Wire Wire Line
-	4200 3650 4300 3650
 Wire Wire Line
 	4200 4100 4200 4250
@@
 Wire Wire Line
 	8200 4050 7750 4050
+Wire Wire Line
+	4200 3650 4450 3650
 $EndSCHEMATC
