File: Hartware_2.0.0/Acon_NTC.sch (KiCad schematic (older format))
At the start: 4 parts, among them P2 CONN_01X02, P3 CONN_01X02

Commit message: primer trabajo de codificacion
Parts:
- P2, P3: footprint Pin_Headers:Pin_Header_Straight_1x02 -> Connector_PinHeader_2.54mm:PinHeader_2x01_P2.54mm_Vertical; symbol D21_2550-rescue:Conn_01x02-RESCUE-D21_2550 -> Connector_Generic:Conn_01x02
- R18, R19: footprint Resistors_SMD:R_0805_HandSoldering -> Resistor_SMD:R_0805_2012Metric_Pad1.15x1.50mm_HandSolder; symbol D21_2550-rescue:R-RESCUE-D21_2550 -> Device:R
Connections:
- wire segments 10 -> 12
Changed lines of the file:
@@
 $EndDescr
 $Comp
-L D21_2550-rescue:Conn_01x02-RESCUE-D21_2550 P2
+L Connector_Generic:Conn_01x02 P2
 U 1 1 56D55FD7
-P 3850 2900
-F 0 "P2" H 3850 3050 50  0000 C CNN
-F 1 "CONN_01X02" V 3950 2900 50  0000 C CNN
-F 2 "Pin_Headers:Pin_Header_Straight_1x02" H 3850 2900 50  0001 C CNN
-F 3 "" H 3850 2900 50  0000 C CNN
-	1    3850 2900
+P 3850 2950
+F 0 "P2" H 3850 3100 50  0000 C CNN
+F 1 "CONN_01X02" V 3950 2950 50  0000 C CNN
+F 2 "Connector_PinHeader_2.54mm:PinHeader_2x01_P2.54mm_Vertical" H 3850 2950 50  0001 C CNN
+F 3 "" H 3850 2950 50  0000 C CNN
+	1    3850 2950
 	-1   0    0    1
 $EndComp
 $Comp
-L D21_2550-rescue:Conn_01x02-RESCUE-D21_2550 P3
+L Connector_Generic:Conn_01x02 P3
 U 1 1 56D56090
-P 3850 5050
-F 0 "P3" H 3850 5200 50  0000 C CNN
-F 1 "CONN_01X02" V 3950 5050 50  0000 C CNN
-F 2 "Pin_Headers:Pin_Header_Straight_1x02" H 3850 5050 50  0001 C CNN
-F 3 "" H 3850 5050 50  0000 C CNN
-	1    3850 5050
+P 3850 5100
+F 0 "P3" H 3850 5250 50  0000 C CNN
+F 1 "CONN_01X02" V 3950 5100 50  0000 C CNN
+F 2 "Connector_PinHeader_2.54mm:PinHeader_2x01_P2.54mm_Vertical" H 3850 5100 50  0001 C CNN
+F 3 "" H 3850 5100 50  0000 C CNN
+	1    3850 5100
 	-1   0    0    1
 $EndComp
@@
 T_R
 $Comp
-L D21_2550-rescue:R-RESCUE-D21_2550 R18
+L Device:R R18
 U 1 1 56FD73A4
 P 4100 2100
 F 0 "R18" V 4180 2100 50  0000 C CNN
 F 1 "20k" V 4100 2100 50  0000 C CNN
-F 2 "Resistors_SMD:R_0805_HandSoldering" V 4030 2100 50  0001 C CNN
+F 2 "Resistor_SMD:R_0805_2012Metric_Pad1.15x1.50mm_HandSolder" V 4030 2100 50  0001 C CNN
 F 3 "" H 4100 2100 50  0000 C CNN
 	1    4100 2100
@@
 $EndComp
 $Comp
-L D21_2550-rescue:R-RESCUE-D21_2550 R19
+L Device:R R19
 U 1 1 56FD753F
 P 4100 4500
 F 0 "R19" V 4180 4500 50  0000 C CNN
 F 1 "20k" V 4100 4500 50  0000 C CNN
-F 2 "Resistors_SMD:R_0805_HandSoldering" V 4030 4500 50  0001 C CNN
+F 2 "Resistor_SMD:R_0805_2012Metric_Pad1.15x1.50mm_HandSolder" V 4030 4500 50  0001 C CNN
 F 3 "" H 4100 4500 50  0000 C CNN
 	1    4100 4500
 	1    0    0    -1
 $EndComp
-$Comp
-L GND-RESCUE-D21_2550 #PWR013
-U 1 1 56FD75D4
-P 4100 5450
-F 0 "#PWR013" H 4100 5200 50  0001 C CNN
-F 1 "GND" H 4100 5300 50  0000 C CNN
-F 2 "" H 4100 5450 50  0000 C CNN
-F 3 "" H 4100 5450 50  0000 C CNN
-	1    4100 5450
-	1    0    0    -1
-$EndComp
-$Comp
-L GND-RESCUE-D21_2550 #PWR014
-U 1 1 56FD7654
-P 4100 3350
-F 0 "#PWR014" H 4100 3100 50  0001 C CNN
-F 1 "GND" H 4100 3200 50  0000 C CNN
-F 2 "" H 4100 3350 50  0000 C CNN
-F 3 "" H 4100 3350 50  0000 C CNN
-	1    4100 3350
-	1    0    0    -1
-$EndComp
 Wire Wire Line
-	4050 5000 4350 5000
+	4050 5000 4100 5000
 Wire Wire Line
 	4100 5000 4100 4650
@@
 	4100 2950 4100 3350
 Wire Wire Line
-	4050 2850 4300 2850
+	4050 2850 4100 2850
 Wire Wire Line
 	4100 2850 4100 2250
@@
 Connection ~ 4100 5000
 Connection ~ 4100 2850
+Wire Wire Line
+	4100 5000 4350 5000
+Wire Wire Line
+	4100 2850 4300 2850
+$Comp
+L power:GND #PWR013
+U 1 1 5A80DF5C
+P 4100 3350
+F 0 "#PWR013" H 4100 3100 50  0001 C CNN
+F 1 "GND" H 4105 3177 50  0000 C CNN
+F 2 "" H 4100 3350 50  0001 C CNN
+F 3 "" H 4100 3350 50  0001 C CNN
+	1    4100 3350
+	1    0    0    -1
+$EndComp
+$Comp
+L power:GND #PWR014
+U 1 1 5A80DFC2
+P 4100 5450
+F 0 "#PWR014" H 4100 5200 50  0001 C CNN
+F 1 "GND" H 4105 5277 50  0000 C CNN
+F 2 "" H 4100 5450 50  0001 C CNN
+F 3 "" H 4100 5450 50  0001 C CNN
+	1    4100 5450
+	1    0    0    -1
+$EndComp
 $EndSCHEMATC

Commit message: termino parcial de la version 2
Parts:
- P2: value CONN_01X02 -> TA
- P3: value CONN_01X02 -> TR
- R18, R19: Campo4 (none) -> RG2012P-203-B-T5
Changed lines of the file:
@@
 P 3850 2950
 F 0 "P2" H 3850 3100 50  0000 C CNN
-F 1 "CONN_01X02" V 3950 2950 50  0000 C CNN
+F 1 "TA" V 3950 2950 50  0000 C CNN
 F 2 "Connector_PinHeader_2.54mm:PinHeader_2x01_P2.54mm_Vertical" H 3850 2950 50  0001 C CNN
 F 3 "" H 3850 2950 50  0000 C CNN
@@
 P 3850 5100
 F 0 "P3" H 3850 5250 50  0000 C CNN
-F 1 "CONN_01X02" V 3950 5100 50  0000 C CNN
+F 1 "TR" V 3950 5100 50  0000 C CNN
 F 2 "Connector_PinHeader_2.54mm:PinHeader_2x01_P2.54mm_Vertical" H 3850 5100 50  0001 C CNN
 F 3 "" H 3850 5100 50  0000 C CNN
@@
 F 1 "20k" V 4100 2100 50  0000 C CNN
 F 2 "Resistor_SMD:R_0805_2012Metric_Pad1.15x1.50mm_HandSolder" V 4030 2100 50  0001 C CNN
-F 3 "" H 4100 2100 50  0000 C CNN
+F 3 "http://www.susumu.co.jp/common/pdf/n_catalog_partition01_en.pdf" H 4100 2100 50  0001 C CNN
+F 4 "RG2012P-203-B-T5" V 4100 2100 50  0001 C CNN "Campo4"
 	1    4100 2100
 	1    0    0    -1
@@
 F 1 "20k" V 4100 4500 50  0000 C CNN
 F 2 "Resistor_SMD:R_0805_2012Metric_Pad1.15x1.50mm_HandSolder" V 4030 4500 50  0001 C CNN
-F 3 "" H 4100 4500 50  0000 C CNN
+F 3 "http://www.susumu.co.jp/common/pdf/n_catalog_partition01_en.pdf" H 4100 4500 50  0001 C CNN
+F 4 "RG2012P-203-B-T5" V 4100 4500 50  0001 C CNN "Campo4"
 	1    4100 4500
 	1    0    0    -1

Commit message: finalinzando la placa
Parts:
- removed P2: TA, Connector_PinHeader_2.54mm:PinHeader_2x01_P2.54mm_Vertical, symbol Connector_Generic:Conn_01x02
- removed P3: TR, Connector_PinHeader_2.54mm:PinHeader_2x01_P2.54mm_Vertical, symbol Connector_Generic:Conn_01x02
- added J1: THR, Connector_JST:JST_XH_B04B-XH-A_1x04_P2.50mm_Vertical, symbol Connector_Generic:Conn_01x04
Connections:
- wire segments 12 -> 15
Changed lines of the file:
@@
 Comment4 ""
 $EndDescr
-$Comp
-L Connector_Generic:Conn_01x02 P2
-U 1 1 56D55FD7
-P 3850 2950
-F 0 "P2" H 3850 3100 50  0000 C CNN
-F 1 "TA" V 3950 2950 50  0000 C CNN
-F 2 "Connector_PinHeader_2.54mm:PinHeader_2x01_P2.54mm_Vertical" H 3850 2950 50  0001 C CNN
-F 3 "" H 3850 2950 50  0000 C CNN
-	1    3850 2950
-	-1   0    0    1
-$EndComp
-$Comp
-L Connector_Generic:Conn_01x02 P3
-U 1 1 56D56090
-P 3850 5100
-F 0 "P3" H 3850 5250 50  0000 C CNN
-F 1 "TR" V 3950 5100 50  0000 C CNN
-F 2 "Connector_PinHeader_2.54mm:PinHeader_2x01_P2.54mm_Vertical" H 3850 5100 50  0001 C CNN
-F 3 "" H 3850 5100 50  0000 C CNN
-	1    3850 5100
-	-1   0    0    1
-$EndComp
-Text GLabel 4100 1700 1    60   Input ~ 0
+Text GLabel 5900 3450 1    60   Input ~ 0
 VDD
-Text GLabel 4100 4150 1    60   Input ~ 0
-VDD
-Text HLabel 4300 2850 2    60   Output ~ 0
+Text HLabel 6150 4100 2    60   Output ~ 0
 T_A
-Text HLabel 4350 5000 2    60   Output ~ 0
+Text HLabel 6150 4300 2    60   Output ~ 0
 T_R
 $Comp
 L Device:R R18
 U 1 1 56FD73A4
-P 4100 2100
-F 0 "R18" V 4180 2100 50  0000 C CNN
-F 1 "20k" V 4100 2100 50  0000 C CNN
-F 2 "Resistor_SMD:R_0805_2012Metric_Pad1.15x1.50mm_HandSolder" V 4030 2100 50  0001 C CNN
-F 3 "http://www.susumu.co.jp/common/pdf/n_catalog_partition01_en.pdf" H 4100 2100 50  0001 C CNN
-F 4 "RG2012P-203-B-T5" V 4100 2100 50  0001 C CNN "Campo4"
-	1    4100 2100
+P 5800 3800
+F 0 "R18" V 5880 3800 50  0000 C CNN
+F 1 "20k" V 5800 3800 50  0000 C CNN
+F 2 "Resistor_SMD:R_0805_2012Metric_Pad1.15x1.50mm_HandSolder" V 5730 3800 50  0001 C CNN
+F 3 "http://www.susumu.co.jp/common/pdf/n_catalog_partition01_en.pdf" H 5800 3800 50  0001 C CNN
+F 4 "RG2012P-203-B-T5" V 5800 3800 50  0001 C CNN "Campo4"
+	1    5800 3800
 	1    0    0    -1
 $EndComp
@@
 L Device:R R19
 U 1 1 56FD753F
-P 4100 4500
-F 0 "R19" V 4180 4500 50  0000 C CNN
-F 1 "20k" V 4100 4500 50  0000 C CNN
-F 2 "Resistor_SMD:R_0805_2012Metric_Pad1.15x1.50mm_HandSolder" V 4030 4500 50  0001 C CNN
-F 3 "http://www.susumu.co.jp/common/pdf/n_catalog_partition01_en.pdf" H 4100 4500 50  0001 C CNN
-F 4 "RG2012P-203-B-T5" V 4100 4500 50  0001 C CNN "Campo4"
-	1    4100 4500
+P 6000 3800
+F 0 "R19" V 6080 3800 50  0000 C CNN
+F 1 "20k" V 6000 3800 50  0000 C CNN
+F 2 "Resistor_SMD:R_0805_2012Metric_Pad1.15x1.50mm_HandSolder" V 5930 3800 50  0001 C CNN
+F 3 "http://www.susumu.co.jp/common/pdf/n_catalog_partition01_en.pdf" H 6000 3800 50  0001 C CNN
+F 4 "RG2012P-203-B-T5" V 6000 3800 50  0001 C CNN "Campo4"
+	1    6000 3800
 	1    0    0    -1
 $EndComp
 Wire Wire Line
-	4050 5000 4100 5000
+	6000 4300 6000 3950
 Wire Wire Line
-	4100 5000 4100 4650
+	5800 4200 5800 4400
 Wire Wire Line
-	4050 5100 4100 5100
+	5800 4100 5800 3950
 Wire Wire Line
-	4100 5100 4100 5450
+	5800 3550 5800 3650
+Connection ~ 6000 4300
+Connection ~ 5800 4100
 Wire Wire Line
-	4050 2950 4100 2950
+	6000 4300 6150 4300
 Wire Wire Line
-	4100 2950 4100 3350
-Wire Wire Line
-	4050 2850 4100 2850
-Wire Wire Line
-	4100 2850 4100 2250
-Wire Wire Line
-	4100 1700 4100 1950
-Wire Wire Line
-	4100 4350 4100 4150
-Connection ~ 4100 5000
-Connection ~ 4100 2850
-Wire Wire Line
-	4100 5000 4350 5000
-Wire Wire Line
-	4100 2850 4300 2850
+	5800 4100 6150 4100
 $Comp
 L power:GND #PWR013
 U 1 1 5A80DF5C
-P 4100 3350
-F 0 "#PWR013" H 4100 3100 50  0001 C CNN
-F 1 "GND" H 4105 3177 50  0000 C CNN
-F 2 "" H 4100 3350 50  0001 C CNN
-F 3 "" H 4100 3350 50  0001 C CNN
-	1    4100 3350
+P 5800 4600
+F 0 "#PWR013" H 5800 4350 50  0001 C CNN
+F 1 "GND" H 5805 4427 50  0000 C CNN
+F 2 "" H 5800 4600 50  0001 C CNN
+F 3 "" H 5800 4600 50  0001 C CNN
+	1    5800 4600
 	1    0    0    -1
 $EndComp
 $Comp
-L power:GND #PWR014
-U 1 1 5A80DFC2
-P 4100 5450
-F 0 "#PWR014" H 4100 5200 50  0001 C CNN
-F 1 "GND" H 4105 5277 50  0000 C CNN
-F 2 "" H 4100 5450 50  0001 C CNN
-F 3 "" H 4100 5450 50  0001 C CNN
-	1    4100 5450
-	1    0    0    -1
+L Connector_Generic:Conn_01x04 J1
+U 1 1 5A8A68C2
+P 5350 4300
+F 0 "J1" H 5270 3875 50  0000 C CNN
+F 1 "THR" H 5270 3966 50  0000 C CNN
+F 2 "Connector_JST:JST_XH_B04B-XH-A_1x04_P2.50mm_Vertical" H 5350 4300 50  0001 C CNN
+F 3 "https://www.digikey.com/product-detail/en/jst-sales-america-inc/B4B-XH-A-LF-SN/455-2249-ND/1651047" H 5350 4300 50  0001 C CNN
+F 4 "B4B-XH-A(LF)(SN)" H 5350 4300 50  0001 C CNN "Campo4"
+	1    5350 4300
+	-1   0    0    1
 $EndComp
+Wire Wire Line
+	5550 4100 5800 4100
+Wire Wire Line
+	5550 4200 5800 4200
+Wire Wire Line
+	5550 4300 6000 4300
+Wire Wire Line
+	5550 4400 5800 4400
+Connection ~ 5800 4400
+Wire Wire Line
+	5800 4400 5800 4600
+Wire Wire Line
+	5800 3550 5900 3550
+Wire Wire Line
+	6000 3550 6000 3650
+Wire Wire Line
+	5900 3450 5900 3550
+Connection ~ 5900 3550
+Wire Wire Line
+	5900 3550 6000 3550
 $EndSCHEMATC

Commit message: colocando conector de JST de 90grados
Parts:
- J1: footprint Connector_JST:JST_XH_B04B-XH-A_1x04_P2.50mm_Vertical -> Connector_JST:JST_XH_S04B-XH-A-1_1x04_P2.50mm_Horizontal; Campo4 B4B-XH-A(LF)(SN) -> S4B-XH-A(LF)(SN)
Changed lines of the file:
@@
 F 0 "J1" H 5270 3875 50  0000 C CNN
 F 1 "THR" H 5270 3966 50  0000 C CNN
-F 2 "Connector_JST:JST_XH_B04B-XH-A_1x04_P2.50mm_Vertical" H 5350 4300 50  0001 C CNN
-F 3 "https://www.digikey.com/product-detail/en/jst-sales-america-inc/B4B-XH-A-LF-SN/455-2249-ND/1651047" H 5350 4300 50  0001 C CNN
-F 4 "B4B-XH-A(LF)(SN)" H 5350 4300 50  0001 C CNN "Campo4"
+F 2 "Connector_JST:JST_XH_S04B-XH-A-1_1x04_P2.50mm_Horizontal" H 5350 4300 50  0001 C CNN
+F 3 "http://www.jst-mfg.com/product/pdf/eng/eXH.pdf" H 5350 4300 50  0001 C CNN
+F 4 "S4B-XH-A(LF)(SN)" H 5350 4300 50  0001 C CNN "Campo4"
 	1    5350 4300
 	-1   0    0    1
