File: Hartware_2.0.0/Cerebro.sch (KiCad schematic (older format))
At the start: 15 parts, among them P4 CONN_01X05, U1 PIC18F2550, Y1 4MHZ

Commit message: primer trabajo de codificacion
Parts:
- removed U1: PIC18F2550, Housings_SOIC:SOIC-28_7.5x17.9mm_Pitch1.27mm, symbol D21_2550-rescue:PIC18F2550-RESCUE-D21_2550
- added U1: PIC18F2550-ISO, Package_SOIC:SOIC-28W_7.5x17.9mm_P1.27mm, symbol MCU_Microchip_PIC18:PIC18F2550-ISO
- C2, C3: symbol D21_2550-rescue:C-RESCUE-D21_2550 -> Device:C
- C7: footprint Capacitors_ThroughHole:C_Radial_D5_L11_P2 -> Capacitor_SMD:CP_Elec_3x5.3; symbol D21_2550-rescue:CP1_Small-RESCUE-D21_2550 -> Device:CP1_Small
- D10, D8, D9: footprint LEDs:LED-3MM -> LED_SMD:LED_PLCC-2; symbol D21_2550-rescue:LED_Small-RESCUE-D21_2550 -> Device:LED_Small
- D6: footprint Diodes_SMD:SOD-123 -> Diode_SMD:D_SOD-123; symbol D21_2550-rescue:D-RESCUE-D21_2550 -> Device:D
- D7: symbol D21_2550-rescue:D-RESCUE-D21_2550 -> Device:D
- P4: value CONN_01X05 -> ISCP; footprint Pin_Headers:Pin_Header_Straight_1x05 -> Connector_PinHeader_2.54mm:PinHeader_1x05_P2.54mm_Vertical; symbol D21_2550-rescue:Conn_01x05-RESCUE-D21_2550 -> Connector_Generic:Conn_01x05
- R2, R24, R25, R26: footprint Resistors_SMD:R_0805_HandSoldering -> Resistor_SMD:R_0805_2012Metric_Pad1.15x1.50mm_HandSolder; symbol D21_2550-rescue:R-RESCUE-D21_2550 -> Device:R
- Y1: footprint Crystals:Crystal_HC49-U_Vertical -> Crystal:Crystal_SMD_5032-2Pin_5.0x3.2mm_HandSoldering; symbol D21_2550-rescue:Crystal-RESCUE-D21_2550 -> Device:Crystal
Connections:
- wire segments 85 -> 89

Commit message: modificacion de cartas
Parts:
- C2, C3: footprint Capacitors_SMD:C_0805_HandSoldering -> Capacitor_SMD:C_0805_2012Metric_Pad1.15x1.50mm_HandSolder
- D7: footprint Diodes_SMD:SOD-123 -> Diode_SMD:D_SOD-123
Changed lines of the file:
@@
 F1 "Acon_NTC.sch" 60
 F2 "T_A" O R 4100 2300 60
-F3 "T_R" O R 4100 2150 60
+F3 "T_R" O R 4100 2200 60
 $EndSheet
 Wire Wire Line
-	4100 2150 4400 2150
-Wire Wire Line
-	4400 2150 4400 2600
+	4400 2200 4400 2600
 Wire Wire Line
 	4400 2600 4650 2600
@@
 F 0 "C2" H 1875 4650 50  0000 L CNN
 F 1 "33pf" H 1875 4450 50  0000 L CNN
-F 2 "Capacitors_SMD:C_0805_HandSoldering" H 1888 4400 50  0001 C CNN
+F 2 "Capacitor_SMD:C_0805_2012Metric_Pad1.15x1.50mm_HandSolder" H 1888 4400 50  0001 C CNN
 F 3 "" H 1850 4550 50  0000 C CNN
 	1    1850 4550
@@
 F 0 "C3" H 2375 4650 50  0000 L CNN
 F 1 "33pf" H 2375 4450 50  0000 L CNN
-F 2 "Capacitors_SMD:C_0805_HandSoldering" H 2388 4400 50  0001 C CNN
+F 2 "Capacitor_SMD:C_0805_2012Metric_Pad1.15x1.50mm_HandSolder" H 2388 4400 50  0001 C CNN
 F 3 "" H 2350 4550 50  0000 C CNN
 	1    2350 4550
@@
 F 0 "D7" H 9750 5450 50  0000 C CNN
 F 1 "1N4007" H 9750 5250 50  0000 C CNN
-F 2 "Diodes_SMD:SOD-123" H 9750 5350 50  0001 C CNN
+F 2 "Diode_SMD:D_SOD-123" H 9750 5350 50  0001 C CNN
 F 3 "" H 9750 5350 50  0000 C CNN
 	1    9750 5350
@@
 	5850 2300 5850 2000
 Connection ~ 5850 2000
+Wire Wire Line
+	4400 2200 4100 2200
 $EndSCHEMATC

Commit message: a medio hacer
Parts:
- D10: value D_R -> LED; footprint LED_SMD:LED_PLCC-2 -> LED_SMD:LED_0603_1608Metric_Pad0.67x1.00mm_HandSolder; Campo4 (none) -> 150060BS75000
- D6, D7: value 1N4007 -> 1N4148X-TP; footprint Diode_SMD:D_SOD-123 -> Diode_SMD:D_SOD-523; Campo4 (none) -> 1N4148X-TP
- D8: value D_C -> LED; footprint LED_SMD:LED_PLCC-2 -> LED_SMD:LED_0603_1608Metric_Pad0.67x1.00mm_HandSolder; Campo4 (none) -> 150060BS75000
- D9: value D_V -> LED; footprint LED_SMD:LED_PLCC-2 -> LED_SMD:LED_0603_1608Metric_Pad0.67x1.00mm_HandSolder; Campo4 (none) -> 150060BS75000
- U1: Campo4 (none) -> PIC18F2550-I/SO
- Y1: value 4MHZ -> 20MHZ; footprint Crystal:Crystal_SMD_5032-2Pin_5.0x3.2mm_HandSoldering -> Devices_MSS:Crystal_SMD_ABLS_HC49-SD; Campo4 (none) -> ABLS-20.000MHZ-B2-T
Changed lines of the file:
@@
 P 2100 4150
 F 0 "Y1" H 2100 4300 50  0000 C CNN
-F 1 "4MHZ" H 2100 4000 50  0000 C CNN
-F 2 "Crystal:Crystal_SMD_5032-2Pin_5.0x3.2mm_HandSoldering" H 2100 4150 50  0001 C CNN
-F 3 "" H 2100 4150 50  0000 C CNN
+F 1 "20MHZ" H 2100 4000 50  0000 C CNN
+F 2 "Devices_MSS:Crystal_SMD_ABLS_HC49-SD" H 2100 4150 50  0001 C CNN
+F 3 "http://www.abracon.com/Resonators/abls.pdf" H 2100 4150 50  0001 C CNN
+F 4 "ABLS-20.000MHZ-B2-T" H 2100 4150 50  0001 C CNN "Campo4"
 	1    2100 4150
 	1    0    0    -1
@@
 P 9750 5350
 F 0 "D7" H 9750 5450 50  0000 C CNN
-F 1 "1N4007" H 9750 5250 50  0000 C CNN
-F 2 "Diode_SMD:D_SOD-123" H 9750 5350 50  0001 C CNN
-F 3 "" H 9750 5350 50  0000 C CNN
+F 1 "1N4148X-TP" H 9750 5250 50  0000 C CNN
+F 2 "Diode_SMD:D_SOD-523" H 9750 5350 50  0001 C CNN
+F 3 "http://www.mccsemi.com/up_pdf/1N4148X(SOD-523).PDF" H 9750 5350 50  0001 C CNN
+F 4 "1N4148X-TP" H 9750 5350 50  0001 C CNN "Campo4"
 	1    9750 5350
 	1    0    0    -1
@@
 P 5850 1800
 F 0 "D6" H 5850 1900 50  0000 C CNN
-F 1 "1N4007" H 5850 1700 50  0000 C CNN
-F 2 "Diode_SMD:D_SOD-123" H 5850 1950 50  0001 C CNN
-F 3 "" H 5850 1800 50  0000 C CNN
+F 1 "1N4148X-TP" H 5850 1700 50  0000 C CNN
+F 2 "Diode_SMD:D_SOD-523" H 5850 1950 50  0001 C CNN
+F 3 "http://www.mccsemi.com/up_pdf/1N4148X(SOD-523).PDF" H 5850 1800 50  0001 C CNN
+F 4 "1N4148X-TP" H 5850 1800 50  0001 C CNN "Campo4"
 	1    5850 1800
 	0    -1   -1   0
@@
 P 9150 3850
 F 0 "D10" H 9100 3975 50  0000 L CNN
-F 1 "D_R" H 9100 3750 50  0000 L CNN
-F 2 "LED_SMD:LED_PLCC-2" V 9150 3850 50  0001 C CNN
-F 3 "" V 9150 3850 50  0000 C CNN
+F 1 "LED" H 9100 3750 50  0000 L CNN
+F 2 "LED_SMD:LED_0603_1608Metric_Pad0.67x1.00mm_HandSolder" V 9150 3850 50  0001 C CNN
+F 3 "http://katalog.we-online.de/led/datasheet/150060BS75000.pdf" H 9150 3850 50  0001 C CNN
+F 4 "150060BS75000" H 9150 3850 50  0001 C CNN "Campo4"
 	1    9150 3850
 	0    -1   -1   0
@@
 P 8850 3850
 F 0 "D9" H 8800 3975 50  0000 L CNN
-F 1 "D_V" H 8800 3750 50  0000 L CNN
-F 2 "LED_SMD:LED_PLCC-2" V 8850 3850 50  0001 C CNN
-F 3 "" V 8850 3850 50  0000 C CNN
+F 1 "LED" H 8800 3750 50  0000 L CNN
+F 2 "LED_SMD:LED_0603_1608Metric_Pad0.67x1.00mm_HandSolder" V 8850 3850 50  0001 C CNN
+F 3 "http://katalog.we-online.de/led/datasheet/150060BS75000.pdf" H 8850 3850 50  0001 C CNN
+F 4 "150060BS75000" H 8850 3850 50  0001 C CNN "Campo4"
 	1    8850 3850
 	0    -1   -1   0
@@
 P 8500 3850
 F 0 "D8" H 8450 3975 50  0000 L CNN
-F 1 "D_C" H 8450 3750 50  0000 L CNN
-F 2 "LED_SMD:LED_PLCC-2" V 8500 3850 50  0001 C CNN
-F 3 "" V 8500 3850 50  0000 C CNN
+F 1 "LED" H 8450 3750 50  0000 L CNN
+F 2 "LED_SMD:LED_0603_1608Metric_Pad0.67x1.00mm_HandSolder" V 8500 3850 50  0001 C CNN
+F 3 "http://katalog.we-online.de/led/datasheet/150060BS75000.pdf" H 8500 3850 50  0001 C CNN
+F 4 "150060BS75000" H 8500 3850 50  0001 C CNN "Campo4"
 	1    8500 3850
 	0    -1   -1   0
@@
 F 2 "Package_SOIC:SOIC-28W_7.5x17.9mm_P1.27mm" H 5850 3400 50  0001 C CIN
 F 3 "http://ww1.microchip.com/downloads/en/devicedoc/39632c.pdf" H 5850 2950 50  0001 C CNN
+F 4 "PIC18F2550-I/SO" H 5850 3400 50  0001 C CNN "Campo4"
 	1    5850 3400
 	1    0    0    -1

Commit message: final placa v2
Changed lines of the file:
@@
 Wire Wire Line
 	5850 1650 5850 1500
-Text GLabel 5950 2000 2    60   Input ~ 0
+Text GLabel 6200 2000 2    60   Input ~ 0
 VDDP
 Wire Wire Line
-	5950 2000 5850 2000
+	6200 2000 5850 2000
 $Comp
 L Connector_Generic:Conn_01x05 P4

Commit message: termino parcial de la version 2
Parts:
- C2, C3: Campo4 (none) -> C0805C103K5RACTU
- R2: Campo4 (none) -> ERA-6AEB103V
- R24, R25, R26: Campo4 (none) -> ESR10EZPJ221
Changed lines of the file:
@@
 F 1 "33pf" H 1875 4450 50  0000 L CNN
 F 2 "Capacitor_SMD:C_0805_2012Metric_Pad1.15x1.50mm_HandSolder" H 1888 4400 50  0001 C CNN
-F 3 "" H 1850 4550 50  0000 C CNN
+F 3 "https://search.kemet.com/component-edge/download/datasheet/C0805C103K5RACTU.pdf" H 1850 4550 50  0001 C CNN
+F 4 "C0805C103K5RACTU" H 1850 4550 50  0001 C CNN "Campo4"
 	1    1850 4550
 	1    0    0    -1
@@
 F 1 "33pf" H 2375 4450 50  0000 L CNN
 F 2 "Capacitor_SMD:C_0805_2012Metric_Pad1.15x1.50mm_HandSolder" H 2388 4400 50  0001 C CNN
-F 3 "" H 2350 4550 50  0000 C CNN
+F 3 "https://search.kemet.com/component-edge/download/datasheet/C0805C103K5RACTU.pdf" H 2350 4550 50  0001 C CNN
+F 4 "C0805C103K5RACTU" H 2350 4550 50  0001 C CNN "Campo4"
 	1    2350 4550
 	1    0    0    -1
@@
 F 1 "10k" V 10100 5150 50  0000 C CNN
 F 2 "Resistor_SMD:R_0805_2012Metric_Pad1.15x1.50mm_HandSolder" V 10030 5150 50  0001 C CNN
-F 3 "" H 10100 5150 50  0000 C CNN
+F 3 "https://industrial.panasonic.com/cdbs/www-data/pdf/RDM0000/AOA0000C307.pdf" H 10100 5150 50  0001 C CNN
+F 4 "ERA-6AEB103V" V 10100 5150 50  0001 C CNN "Campo4"
 	1    10100 5150
 	1    0    0    -1
@@
 F 1 "220" V 9150 3450 50  0000 C CNN
 F 2 "Resistor_SMD:R_0805_2012Metric_Pad1.15x1.50mm_HandSolder" V 9080 3450 50  0001 C CNN
-F 3 "" H 9150 3450 50  0000 C CNN
+F 3 "http://www.rohm.com/web/global/datasheet/ESR01MZPF/esr-e" H 9150 3450 50  0001 C CNN
+F 4 "ESR10EZPJ221" V 9150 3450 50  0001 C CNN "Campo4"
 	1    9150 3450
 	1    0    0    -1
@@
 F 1 "220" V 8850 3450 50  0000 C CNN
 F 2 "Resistor_SMD:R_0805_2012Metric_Pad1.15x1.50mm_HandSolder" V 8780 3450 50  0001 C CNN
-F 3 "" H 8850 3450 50  0000 C CNN
+F 3 "http://www.rohm.com/web/global/datasheet/ESR01MZPF/esr-e" H 8850 3450 50  0001 C CNN
+F 4 "ESR10EZPJ221" V 8850 3450 50  0001 C CNN "Campo4"
 	1    8850 3450
 	1    0    0    -1
@@
 F 1 "220" V 8500 3450 50  0000 C CNN
 F 2 "Resistor_SMD:R_0805_2012Metric_Pad1.15x1.50mm_HandSolder" V 8430 3450 50  0001 C CNN
-F 3 "" H 8500 3450 50  0000 C CNN
+F 3 "http://www.rohm.com/web/global/datasheet/ESR01MZPF/esr-e" H 8500 3450 50  0001 C CNN
+F 4 "ESR10EZPJ221" V 8500 3450 50  0001 C CNN "Campo4"
 	1    8500 3450
 	1    0    0    -1

Commit message: agregando BOM
Parts:
- C7: footprint Capacitor_SMD:CP_Elec_3x5.3 -> Capacitor_SMD:CP_Elec_4x5.3; Campo4 (none) -> EEE-1CA100SR
Changed lines of the file:
@@
 F 0 "C7" H 10110 5620 50  0000 L CNN
 F 1 "10uf" H 10110 5470 50  0000 L CNN
-F 2 "Capacitor_SMD:CP_Elec_3x5.3" H 10100 5550 50  0001 C CNN
-F 3 "" H 10100 5550 50  0000 C CNN
+F 2 "Capacitor_SMD:CP_Elec_4x5.3" H 10100 5550 50  0001 C CNN
+F 3 "https://industrial.panasonic.com/cdbs/www-data/pdf/RDE0000/ABA0000C1145.pdf" H 10100 5550 50  0001 C CNN
+F 4 "EEE-1CA100SR" H 10100 5550 50  0001 C CNN "Campo4"
 	1    10100 5550
 	1    0    0    -1

Commit message: lista por hacer
Parts:
- removed C7: 10uf, Capacitor_SMD:CP_Elec_4x5.3, symbol Device:CP1_Small
- removed D6, D7: 1N4148X-TP, Diode_SMD:D_SOD-523, symbol Device:D
- added JP1: pgm, Connector_PinHeader_2.54mm:PinHeader_1x02_P2.54mm_Vertical, symbol Device:Jumper_NC_Small
Connections:
- wire segments 89 -> 86
Changed lines of the file:
@@
 F5 "-" O R 4100 3100 60
 $EndSheet
-Text GLabel 5850 1500 1    60   Output ~ 0
+Text GLabel 5850 1150 1    60   Output ~ 0
 VDD
-Wire Wire Line
-	5850 1950 5850 2000
 Wire Wire Line
 	7050 3200 9150 3200
@@
 Text GLabel 4550 3300 0    51   BiDi ~ 0
 K2
-Text GLabel 10100 4900 1    60   Input ~ 0
-VDD
-Wire Wire Line
-	10100 4900 10100 5000
-Wire Wire Line
-	10100 5300 10100 5350
 $Comp
 L Device:Crystal Y1
@@
 Wire Wire Line
 	1850 3950 1850 4150
-$Comp
-L Device:R R2
-U 1 1 56FD5F81
-P 10100 5150
-F 0 "R2" V 10180 5150 50  0000 C CNN
-F 1 "10k" V 10100 5150 50  0000 C CNN
-F 2 "Resistor_SMD:R_0805_2012Metric_Pad1.15x1.50mm_HandSolder" V 10030 5150 50  0001 C CNN
-F 3 "https://industrial.panasonic.com/cdbs/www-data/pdf/RDM0000/AOA0000C307.pdf" H 10100 5150 50  0001 C CNN
-F 4 "ERA-6AEB103V" V 10100 5150 50  0001 C CNN "Campo4"
-	1    10100 5150
-	1    0    0    -1
-$EndComp
-$Comp
-L Device:CP1_Small C7
-U 1 1 56FF296D
-P 10100 5550
-F 0 "C7" H 10110 5620 50  0000 L CNN
-F 1 "10uf" H 10110 5470 50  0000 L CNN
-F 2 "Capacitor_SMD:CP_Elec_4x5.3" H 10100 5550 50  0001 C CNN
-F 3 "https://industrial.panasonic.com/cdbs/www-data/pdf/RDE0000/ABA0000C1145.pdf" H 10100 5550 50  0001 C CNN
-F 4 "EEE-1CA100SR" H 10100 5550 50  0001 C CNN "Campo4"
-	1    10100 5550
-	1    0    0    -1
-$EndComp
-Connection ~ 10100 5350
-Wire Wire Line
-	10100 5700 10100 5650
-$Comp
-L Device:D D7
-U 1 1 56FF6C44
-P 9750 5350
-F 0 "D7" H 9750 5450 50  0000 C CNN
-F 1 "1N4148X-TP" H 9750 5250 50  0000 C CNN
-F 2 "Diode_SMD:D_SOD-523" H 9750 5350 50  0001 C CNN
-F 3 "http://www.mccsemi.com/up_pdf/1N4148X(SOD-523).PDF" H 9750 5350 50  0001 C CNN
-F 4 "1N4148X-TP" H 9750 5350 50  0001 C CNN "Campo4"
-	1    9750 5350
-	1    0    0    -1
-$EndComp
-Wire Wire Line
-	9600 5350 9450 5350
-Text GLabel 9450 5350 0    60   Output ~ 0
-VPP
-$Comp
-L Device:D D6
-U 1 1 56FFEF97
-P 5850 1800
-F 0 "D6" H 5850 1900 50  0000 C CNN
-F 1 "1N4148X-TP" H 5850 1700 50  0000 C CNN
-F 2 "Diode_SMD:D_SOD-523" H 5850 1950 50  0001 C CNN
-F 3 "http://www.mccsemi.com/up_pdf/1N4148X(SOD-523).PDF" H 5850 1800 50  0001 C CNN
-F 4 "1N4148X-TP" H 5850 1800 50  0001 C CNN "Campo4"
-	1    5850 1800
-	0    -1   -1   0
-$EndComp
-Wire Wire Line
-	5850 1650 5850 1500
 Text GLabel 6200 2000 2    60   Input ~ 0
 VDDP
-Wire Wire Line
-	6200 2000 5850 2000
 $Comp
 L Connector_Generic:Conn_01x05 P4
@@
 Text GLabel 4550 5000 3    60   Input ~ 0
 PGD
-Wire Wire Line
-	9900 5350 10100 5350
 $Comp
 L Device:R R26
@@
 	2100 4800 2350 4800
 Wire Wire Line
-	10100 5350 10100 5450
-Wire Wire Line
 	8850 4100 9150 4100
 Wire Wire Line
@@
 $EndComp
 $Comp
-L power:GND #PWR06
-U 1 1 5A7B6D43
-P 10100 5700
-F 0 "#PWR06" H 10100 5450 50  0001 C CNN
-F 1 "GND" H 10105 5527 50  0000 C CNN
-F 2 "" H 10100 5700 50  0001 C CNN
-F 3 "" H 10100 5700 50  0001 C CNN
-	1    10100 5700
-	1    0    0    -1
-$EndComp
-$Comp
 L power:GND #PWR04
 U 1 1 5A7B6F79
@@
 Wire Wire Line
 	4650 3300 4550 3300
-Text GLabel 7350 3600 2    60   Input ~ 0
+Text GLabel 7650 3600 2    60   Input ~ 0
 VPP
-Wire Wire Line
-	7350 3600 7050 3600
 NoConn ~ 7050 3400
 Wire Wire Line
@@
 Wire Wire Line
 	4400 2200 4100 2200
+Wire Wire Line
+	7400 3550 7400 3600
+Wire Wire Line
+	7050 3600 7400 3600
+Wire Wire Line
+	7650 3600 7400 3600
+Connection ~ 7400 3600
+$Comp
+L Device:Jumper_NC_Small JP1
+U 1 1 5A93DA15
+P 5850 1600
+F 0 "JP1" V 5804 1675 50  0000 L CNN
+F 1 "pgm" V 5895 1675 50  0000 L CNN
+F 2 "Connector_PinHeader_2.54mm:PinHeader_1x02_P2.54mm_Vertical" H 5850 1600 50  0001 C CNN
+F 3 "~" H 5850 1600 50  0001 C CNN
+	1    5850 1600
+	0    1    1    0
+$EndComp
+Wire Wire Line
+	6200 2000 5850 2000
+Wire Wire Line
+	5850 1700 5850 2000
+$Comp
+L Device:R R2
+U 1 1 56FD5F81
+P 7400 3400
+F 0 "R2" V 7480 3400 50  0000 C CNN
+F 1 "10k" V 7400 3400 50  0000 C CNN
+F 2 "Resistor_SMD:R_0805_2012Metric_Pad1.15x1.50mm_HandSolder" V 7330 3400 50  0001 C CNN
+F 3 "https://industrial.panasonic.com/cdbs/www-data/pdf/RDM0000/AOA0000C307.pdf" H 7400 3400 50  0001 C CNN
+F 4 "ERA-6AEB103V" V 7400 3400 50  0001 C CNN "Campo4"
+	1    7400 3400
+	1    0    0    -1
+$EndComp
+Wire Wire Line
+	5850 1150 5850 1500
+Text GLabel 7400 2850 1    60   Output ~ 0
+VDD
+Wire Wire Line
+	7400 2850 7400 3250
 $EndSCHEMATC
