File: Hartware_2.0.0/OutTriac.sch (KiCad schematic (older format))
At the start: 19 parts, among them P1 CONN_01X05, U2 MOC3021M, U3 MOC3021M, U4 MOC3021M, U5 MAC97A6, U6 MAC97A6, U7 MAC97A6

Commit message: primer trabajo de codificacion
Parts:
- C4, C5, C6: footprint Capacitors_ThroughHole:C_Disc_D6_P5 -> Capacitor_THT:C_Disc_D9.0mm_W2.5mm_P5.00mm; symbol D21_2550-rescue:C-RESCUE-D21_2550 -> Device:C
- P1: footprint Terminal_Blocks:TerminalBlock_Pheonix_MKDS1.5-5pol -> Connector_Molex:Molex_Micro-Fit_3.0_43650-0515_1x05_P3.00mm_Vertical; symbol D21_2550-rescue:Conn_01x05-RESCUE-D21_2550 -> Connector_Generic:Conn_01x05
- R10, R11, R9: footprint Resistors_ThroughHole:Resistor_Horizontal_RM10mm -> Resistor_THT:R_Axial_DIN0309_L9.0mm_D3.2mm_P12.70mm_Horizontal; symbol D21_2550-rescue:R-RESCUE-D21_2550 -> Device:R
- R3, R4, R5: footprint Resistors_SMD:R_0805_HandSoldering -> Resistor_SMD:R_0805_2012Metric_Pad1.15x1.50mm_HandSolder; symbol D21_2550-rescue:R-RESCUE-D21_2550 -> Device:R
- R6, R7, R8: footprint Resistors_ThroughHole:Resistor_Horizontal_RM10mm -> Resistor_SMD:R_0805_2012Metric_Pad1.15x1.50mm_HandSolder; symbol D21_2550-rescue:R-RESCUE-D21_2550 -> Device:R
- U2, U3, U4: value MOC3021M -> MOC3063S-TA1; footprint Housings_DIP:DIP-6_W7.62mm_LongPads -> Package_SOIC:SO-6_4.4x3.6mm_P1.27mm; symbol MOC3021M-RESCUE-D21_2550 -> Relay_SolidState:MOC3021M; Campo4 (none) -> MOC3063S-TA1
- U5, U6, U7: value MAC97A6 -> Z0103MN 5AA4; footprint TO_SOT_Packages_THT:TO-92_Inline_Narrow_Oval -> Package_TO_SOT_SMD:SOT-223; symbol MAC97A6 -> Device:Q_TRIAC_A1GA2; Campo4 (none) -> Z0103MN 5AA4
Connections:
- wire segments 53 -> 62

Commit message: modificacion de cartas
Parts:
- P1: value CONN_01X05 -> POWER I/O
- U2, U3, U4: footprint Package_SOIC:SO-6_4.4x3.6mm_P1.27mm -> Devices_MSS:MOC306X
- U5, U6, U7: symbol Device:Q_TRIAC_A1GA2 -> Device:Q_TRIAC_A1A2G
Changed lines of the file:
@@
 P 8250 4200
 F 0 "P1" H 8250 4550 50  0000 C CNN
-F 1 "CONN_01X05" V 8350 4200 50  0000 C CNN
+F 1 "POWER I/O" V 8350 4200 50  0000 C CNN
 F 2 "Connector_Molex:Molex_Micro-Fit_3.0_43650-0515_1x05_P3.00mm_Vertical" H 8250 4200 50  0001 C CNN
 F 3 "" H 8250 4200 50  0000 C CNN
@@
 	4550 5800 5000 5800
 $Comp
-L Device:Q_TRIAC_A1GA2 U5
+L Device:Q_TRIAC_A1A2G U5
 U 1 1 56E01680
 P 5000 2500
@@
 $EndComp
 $Comp
-L Device:Q_TRIAC_A1GA2 U6
+L Device:Q_TRIAC_A1A2G U6
 U 1 1 56E01A0B
 P 5000 4500
@@
 $EndComp
 $Comp
-L Device:Q_TRIAC_A1GA2 U7
+L Device:Q_TRIAC_A1A2G U7
 U 1 1 56E01C28
 P 5000 6350
@@
 F 0 "U2" H 3340 2690 50  0000 L CNN
 F 1 "MOC3063S-TA1" H 3550 2700 50  0000 L CNN
-F 2 "Package_SOIC:SO-6_4.4x3.6mm_P1.27mm" H 3350 2300 50  0001 L CIN
+F 2 "Devices_MSS:MOC306X" H 3350 2300 50  0001 L CIN
 F 3 "http://optoelectronics.liteon.com/upload/download/DS70-2001-026/MOC306X%20series%20201606.pdf" H 3525 2500 50  0001 L CNN
 F 4 "MOC3063S-TA1" H 3550 2500 50  0001 C CNN "Campo4"
@@
 F 0 "U3" H 3340 4690 50  0000 L CNN
 F 1 "MOC3063S-TA1" H 3550 4700 50  0000 L CNN
-F 2 "Package_SOIC:SO-6_4.4x3.6mm_P1.27mm" H 3350 4300 50  0001 L CIN
+F 2 "Devices_MSS:MOC306X" H 3350 4300 50  0001 L CIN
 F 3 "http://optoelectronics.liteon.com/upload/download/DS70-2001-026/MOC306X%20series%20201606.pdf" H 3525 4500 50  0001 L CNN
 F 4 "MOC3063S-TA1" H 3550 4500 50  0001 C CNN "Campo4"
@@
 F 0 "U4" H 3340 6540 50  0000 L CNN
 F 1 "MOC3063S-TA1" H 3550 6550 50  0000 L CNN
-F 2 "Package_SOIC:SO-6_4.4x3.6mm_P1.27mm" H 3350 6150 50  0001 L CIN
+F 2 "Devices_MSS:MOC306X" H 3350 6150 50  0001 L CIN
 F 3 "http://optoelectronics.liteon.com/upload/download/DS70-2001-026/MOC306X%20series%20201606.pdf" H 3525 6350 50  0001 L CNN
 F 4 "MOC3063S-TA1" H 3550 6350 50  0001 C CNN "Campo4"

Commit message: a medio hacer
Parts:
- C4, C5, C6: value 100nf -> 100nF; footprint Capacitor_THT:C_Disc_D9.0mm_W2.5mm_P5.00mm -> Capacitor_SMD:C_2225_5664Metric_Pad1.78x6.70mm_HandSolder
- P1: footprint Connector_Molex:Molex_Micro-Fit_3.0_43650-0515_1x05_P3.00mm_Vertical -> TerminalBlock:TerminalBlock_bornier-5_P5.08mm
- R10, R11, R9: footprint Resistor_THT:R_Axial_DIN0309_L9.0mm_D3.2mm_P12.70mm_Horizontal -> Resistor_SMD:R_1210_3225Metric_Pad1.24x2.70mm_HandSolder
- U5, U6, U7: footprint Package_TO_SOT_SMD:SOT-223 -> Devices_MSS:SOT-223-Z01
Changed lines of the file:
@@
 F 0 "P1" H 8250 4550 50  0000 C CNN
 F 1 "POWER I/O" V 8350 4200 50  0000 C CNN
-F 2 "Connector_Molex:Molex_Micro-Fit_3.0_43650-0515_1x05_P3.00mm_Vertical" H 8250 4200 50  0001 C CNN
+F 2 "TerminalBlock:TerminalBlock_bornier-5_P5.08mm" H 8250 4200 50  0001 C CNN
 F 3 "" H 8250 4200 50  0000 C CNN
 	1    8250 4200
@@
 F 0 "U5" H 5129 2553 60  0000 L CNN
 F 1 "Z0103MN 5AA4" H 5129 2447 60  0000 L CNN
-F 2 "Package_TO_SOT_SMD:SOT-223" H 4950 2200 60  0001 C CNN
+F 2 "Devices_MSS:SOT-223-Z01" H 4950 2200 60  0001 C CNN
 F 3 "http://www.st.com/content/ccc/resource/technical/document/datasheet/af/ee/c1/7b/df/8a/46/d7/CD00002268.pdf/files/CD00002268.pdf/jcr:content/translations/en.CD00002268.pdf" H 4950 2100 60  0001 C CNN
 F 4 "Z0103MN 5AA4" H 5000 2500 50  0001 C CNN "Campo4"
@@
 F 0 "U6" H 5129 4553 60  0000 L CNN
 F 1 "Z0103MN 5AA4" H 5129 4447 60  0000 L CNN
-F 2 "Package_TO_SOT_SMD:SOT-223" H 4950 4200 60  0001 C CNN
+F 2 "Devices_MSS:SOT-223-Z01" H 4950 4200 60  0001 C CNN
 F 3 "http://www.st.com/content/ccc/resource/technical/document/datasheet/af/ee/c1/7b/df/8a/46/d7/CD00002268.pdf/files/CD00002268.pdf/jcr:content/translations/en.CD00002268.pdf" H 4950 4100 60  0001 C CNN
 F 4 "Z0103MN 5AA4" H 5000 4500 50  0001 C CNN "Campo4"
@@
 F 0 "U7" H 5129 6403 60  0000 L CNN
 F 1 "Z0103MN 5AA4" H 5129 6297 60  0000 L CNN
-F 2 "Package_TO_SOT_SMD:SOT-223" H 4950 6050 60  0001 C CNN
+F 2 "Devices_MSS:SOT-223-Z01" H 4950 6050 60  0001 C CNN
 F 3 "http://www.st.com/content/ccc/resource/technical/document/datasheet/af/ee/c1/7b/df/8a/46/d7/CD00002268.pdf/files/CD00002268.pdf/jcr:content/translations/en.CD00002268.pdf" H 4950 5950 60  0001 C CNN
 F 4 "Z0103MN 5AA4" H 5000 6350 50  0001 C CNN "Campo4"
@@
 F 0 "R9" V 5630 2300 50  0000 C CNN
 F 1 "100" V 5550 2300 50  0000 C CNN
-F 2 "Resistor_THT:R_Axial_DIN0309_L9.0mm_D3.2mm_P12.70mm_Horizontal" V 5480 2300 50  0001 C CNN
+F 2 "Resistor_SMD:R_1210_3225Metric_Pad1.24x2.70mm_HandSolder" V 5480 2300 50  0001 C CNN
 F 3 "" H 5550 2300 50  0000 C CNN
 	1    5550 2300
@@
 F 0 "R10" V 5630 4300 50  0000 C CNN
 F 1 "100" V 5550 4300 50  0000 C CNN
-F 2 "Resistor_THT:R_Axial_DIN0309_L9.0mm_D3.2mm_P12.70mm_Horizontal" V 5480 4300 50  0001 C CNN
+F 2 "Resistor_SMD:R_1210_3225Metric_Pad1.24x2.70mm_HandSolder" V 5480 4300 50  0001 C CNN
 F 3 "" H 5550 4300 50  0000 C CNN
 	1    5550 4300
@@
 F 0 "R11" V 5630 6150 50  0000 C CNN
 F 1 "100" V 5550 6150 50  0000 C CNN
-F 2 "Resistor_THT:R_Axial_DIN0309_L9.0mm_D3.2mm_P12.70mm_Horizontal" V 5480 6150 50  0001 C CNN
+F 2 "Resistor_SMD:R_1210_3225Metric_Pad1.24x2.70mm_HandSolder" V 5480 6150 50  0001 C CNN
 F 3 "" H 5550 6150 50  0000 C CNN
 	1    5550 6150
@@
 AR Path="/56D4C343/56D4C3A8/56FDEE79" Ref="C6"  Part="1"
 F 0 "C6" H 5575 6750 50  0000 L CNN
-F 1 "100nf" H 5575 6550 50  0000 L CNN
-F 2 "Capacitor_THT:C_Disc_D9.0mm_W2.5mm_P5.00mm" H 5588 6500 50  0001 C CNN
+F 1 "100nF" H 5575 6550 50  0000 L CNN
+F 2 "Capacitor_SMD:C_2225_5664Metric_Pad1.78x6.70mm_HandSolder" H 5588 6500 50  0001 C CNN
 F 3 "" H 5550 6650 50  0000 C CNN
 	1    5550 6650
@@
 AR Path="/56D4C343/56D4C3A8/56FDF00C" Ref="C5"  Part="1"
 F 0 "C5" H 5575 4900 50  0000 L CNN
-F 1 "100nf" H 5575 4700 50  0000 L CNN
-F 2 "Capacitor_THT:C_Disc_D9.0mm_W2.5mm_P5.00mm" H 5588 4650 50  0001 C CNN
+F 1 "100nF" H 5575 4700 50  0000 L CNN
+F 2 "Capacitor_SMD:C_2225_5664Metric_Pad1.78x6.70mm_HandSolder" H 5588 4650 50  0001 C CNN
 F 3 "" H 5550 4800 50  0000 C CNN
 	1    5550 4800
@@
 AR Path="/56D4C343/56D4C3A8/56FDF295" Ref="C4"  Part="1"
 F 0 "C4" H 5575 2900 50  0000 L CNN
-F 1 "100nf" H 5575 2700 50  0000 L CNN
-F 2 "Capacitor_THT:C_Disc_D9.0mm_W2.5mm_P5.00mm" H 5588 2650 50  0001 C CNN
+F 1 "100nF" H 5575 2700 50  0000 L CNN
+F 2 "Capacitor_SMD:C_2225_5664Metric_Pad1.78x6.70mm_HandSolder" H 5588 2650 50  0001 C CNN
 F 3 "" H 5550 2800 50  0000 C CNN
 	1    5550 2800

Commit message: final placa v2
Parts:
- C4, C5, C6: footprint Capacitor_SMD:C_2225_5664Metric_Pad1.78x6.70mm_HandSolder -> Capacitor_SMD:C_1206_3216Metric_Pad1.24x1.80mm_HandSolder; Campo4 (none) -> GRM31CR72E104KW03L
Changed lines of the file:
@@
 F 0 "C6" H 5575 6750 50  0000 L CNN
 F 1 "100nF" H 5575 6550 50  0000 L CNN
-F 2 "Capacitor_SMD:C_2225_5664Metric_Pad1.78x6.70mm_HandSolder" H 5588 6500 50  0001 C CNN
-F 3 "" H 5550 6650 50  0000 C CNN
+F 2 "Capacitor_SMD:C_1206_3216Metric_Pad1.24x1.80mm_HandSolder" H 5588 6500 50  0001 C CNN
+F 3 "https://search.murata.co.jp/Ceramy/image/img/A01X/G101/ENG/GRM31CR72E104KW03-01.pdf" H 5550 6650 50  0001 C CNN
+F 4 "GRM31CR72E104KW03L" H 5550 6650 50  0001 C CNN "Campo4"
 	1    5550 6650
 	1    0    0    -1
@@
 F 0 "C5" H 5575 4900 50  0000 L CNN
 F 1 "100nF" H 5575 4700 50  0000 L CNN
-F 2 "Capacitor_SMD:C_2225_5664Metric_Pad1.78x6.70mm_HandSolder" H 5588 4650 50  0001 C CNN
-F 3 "" H 5550 4800 50  0000 C CNN
+F 2 "Capacitor_SMD:C_1206_3216Metric_Pad1.24x1.80mm_HandSolder" H 5588 4650 50  0001 C CNN
+F 3 "https://search.murata.co.jp/Ceramy/image/img/A01X/G101/ENG/GRM31CR72E104KW03-01.pdf" H 5550 4800 50  0001 C CNN
+F 4 "GRM31CR72E104KW03L" H 5550 4800 50  0001 C CNN "Campo4"
 	1    5550 4800
 	1    0    0    -1
@@
 F 0 "C4" H 5575 2900 50  0000 L CNN
 F 1 "100nF" H 5575 2700 50  0000 L CNN
-F 2 "Capacitor_SMD:C_2225_5664Metric_Pad1.78x6.70mm_HandSolder" H 5588 2650 50  0001 C CNN
-F 3 "" H 5550 2800 50  0000 C CNN
+F 2 "Capacitor_SMD:C_1206_3216Metric_Pad1.24x1.80mm_HandSolder" H 5588 2650 50  0001 C CNN
+F 3 "https://search.murata.co.jp/Ceramy/image/img/A01X/G101/ENG/GRM31CR72E104KW03-01.pdf" H 5550 2800 50  0001 C CNN
+F 4 "GRM31CR72E104KW03L" H 5550 2800 50  0001 C CNN "Campo4"
 	1    5550 2800
 	1    0    0    -1

Commit message: termino parcial de la version 2
Parts:
- P1: Campo4 (none) -> 282836-5
- R10, R11, R9: Campo4 (none) -> ERA-6AEB101V
- R3, R4, R5, R6, R7, R8: Campo4 (none) -> ESR10EZPJ331
Changed lines of the file:
@@
 F 1 "POWER I/O" V 8350 4200 50  0000 C CNN
 F 2 "TerminalBlock:TerminalBlock_bornier-5_P5.08mm" H 8250 4200 50  0001 C CNN
-F 3 "" H 8250 4200 50  0000 C CNN
+F 3 "http://www.te.com/commerce/DocumentDelivery/DDEController?Action=srchrtrv&DocNm=282836&DocType=Customer+Drawing&DocLang=English" H 8250 4200 50  0001 C CNN
+F 4 "282836-5" H 8250 4200 50  0001 C CNN "Campo4"
 	1    8250 4200
 	1    0    0    -1
@@
 CO
 Connection ~ 5550 1950
-Text GLabel 7900 4100 0    60   Output ~ 0
+Text GLabel 7900 4300 0    60   Output ~ 0
 RE
 Text GLabel 7650 4200 0    60   Output ~ 0
 VE
-Text GLabel 7900 4300 0    60   Output ~ 0
+Text GLabel 7900 4100 0    60   Output ~ 0
 CO
 Wire Wire Line
@@
 F 1 "330" V 3150 2900 50  0000 C CNN
 F 2 "Resistor_SMD:R_0805_2012Metric_Pad1.15x1.50mm_HandSolder" V 3080 2900 50  0001 C CNN
-F 3 "" H 3150 2900 50  0000 C CNN
+F 3 "http://www.rohm.com/web/global/datasheet/ESR01MZPF/esr-e" H 3150 2900 50  0001 C CNN
+F 4 "ESR10EZPJ331" V 3150 2900 50  0001 C CNN "Campo4"
 	1    3150 2900
 	1    0    0    -1
@@
 F 1 "330" V 4400 1950 50  0000 C CNN
 F 2 "Resistor_SMD:R_0805_2012Metric_Pad1.15x1.50mm_HandSolder" V 4330 1950 50  0001 C CNN
-F 3 "" H 4400 1950 50  0000 C CNN
+F 3 "http://www.rohm.com/web/global/datasheet/ESR01MZPF/esr-e" H 4400 1950 50  0001 C CNN
+F 4 "ESR10EZPJ331" V 4400 1950 50  0001 C CNN "Campo4"
 	1    4400 1950
 	0    1    1    0
@@
 F 1 "100" V 5550 2300 50  0000 C CNN
 F 2 "Resistor_SMD:R_1210_3225Metric_Pad1.24x2.70mm_HandSolder" V 5480 2300 50  0001 C CNN
-F 3 "" H 5550 2300 50  0000 C CNN
+F 3 "https://industrial.panasonic.com/cdbs/www-data/pdf/RDM0000/AOA0000C307.pdf" H 5550 2300 50  0001 C CNN
+F 4 "ERA-6AEB101V" V 5550 2300 50  0001 C CNN "Campo4"
 	1    5550 2300
 	1    0    0    -1
@@
 F 1 "100" V 5550 4300 50  0000 C CNN
 F 2 "Resistor_SMD:R_1210_3225Metric_Pad1.24x2.70mm_HandSolder" V 5480 4300 50  0001 C CNN
-F 3 "" H 5550 4300 50  0000 C CNN
+F 3 "https://industrial.panasonic.com/cdbs/www-data/pdf/RDM0000/AOA0000C307.pdf" H 5550 4300 50  0001 C CNN
+F 4 "ERA-6AEB101V" V 5550 4300 50  0001 C CNN "Campo4"
 	1    5550 4300
 	1    0    0    -1
@@
 F 1 "330" V 4400 3950 50  0000 C CNN
 F 2 "Resistor_SMD:R_0805_2012Metric_Pad1.15x1.50mm_HandSolder" V 4330 3950 50  0001 C CNN
-F 3 "" H 4400 3950 50  0000 C CNN
+F 3 "http://www.rohm.com/web/global/datasheet/ESR01MZPF/esr-e" H 4400 3950 50  0001 C CNN
+F 4 "ESR10EZPJ331" V 4400 3950 50  0001 C CNN "Campo4"
 	1    4400 3950
 	0    1    1    0
@@
 F 1 "330" V 3150 4900 50  0000 C CNN
 F 2 "Resistor_SMD:R_0805_2012Metric_Pad1.15x1.50mm_HandSolder" V 3080 4900 50  0001 C CNN
-F 3 "" H 3150 4900 50  0000 C CNN
+F 3 "http://www.rohm.com/web/global/datasheet/ESR01MZPF/esr-e" H 3150 4900 50  0001 C CNN
+F 4 "ESR10EZPJ331" V 3150 4900 50  0001 C CNN "Campo4"
 	1    3150 4900
 	1    0    0    -1
@@
 F 1 "100" V 5550 6150 50  0000 C CNN
 F 2 "Resistor_SMD:R_1210_3225Metric_Pad1.24x2.70mm_HandSolder" V 5480 6150 50  0001 C CNN
-F 3 "" H 5550 6150 50  0000 C CNN
+F 3 "https://industrial.panasonic.com/cdbs/www-data/pdf/RDM0000/AOA0000C307.pdf" H 5550 6150 50  0001 C CNN
+F 4 "ERA-6AEB101V" V 5550 6150 50  0001 C CNN "Campo4"
 	1    5550 6150
 	1    0    0    -1
@@
 F 1 "330" V 4400 5800 50  0000 C CNN
 F 2 "Resistor_SMD:R_0805_2012Metric_Pad1.15x1.50mm_HandSolder" V 4330 5800 50  0001 C CNN
-F 3 "" H 4400 5800 50  0000 C CNN
+F 3 "http://www.rohm.com/web/global/datasheet/ESR01MZPF/esr-e" H 4400 5800 50  0001 C CNN
+F 4 "ESR10EZPJ331" V 4400 5800 50  0001 C CNN "Campo4"
 	1    4400 5800
 	0    1    1    0
@@
 F 1 "330" V 3150 6750 50  0000 C CNN
 F 2 "Resistor_SMD:R_0805_2012Metric_Pad1.15x1.50mm_HandSolder" V 3080 6750 50  0001 C CNN
-F 3 "" H 3150 6750 50  0000 C CNN
+F 3 "http://www.rohm.com/web/global/datasheet/ESR01MZPF/esr-e" H 3150 6750 50  0001 C CNN
+F 4 "ESR10EZPJ331" V 3150 6750 50  0001 C CNN "Campo4"
 	1    3150 6750
 	1    0    0    -1
@@
 U 1 1 570033F9
 P 3550 2500
-F 0 "U2" H 3340 2690 50  0000 L CNN
-F 1 "MOC3063S-TA1" H 3550 2700 50  0000 L CNN
+F 0 "U2" H 3550 2825 50  0000 C CNN
+F 1 "MOC3063S-TA1" H 3550 2734 50  0000 C CNN
 F 2 "Devices_MSS:MOC306X" H 3350 2300 50  0001 L CIN
 F 3 "http://optoelectronics.liteon.com/upload/download/DS70-2001-026/MOC306X%20series%20201606.pdf" H 3525 2500 50  0001 L CNN
@@
 U 1 1 57004250
 P 3550 4500
-F 0 "U3" H 3340 4690 50  0000 L CNN
-F 1 "MOC3063S-TA1" H 3550 4700 50  0000 L CNN
+F 0 "U3" H 3550 4825 50  0000 C CNN
+F 1 "MOC3063S-TA1" H 3550 4734 50  0000 C CNN
 F 2 "Devices_MSS:MOC306X" H 3350 4300 50  0001 L CIN
 F 3 "http://optoelectronics.liteon.com/upload/download/DS70-2001-026/MOC306X%20series%20201606.pdf" H 3525 4500 50  0001 L CNN
@@
 U 1 1 57004690
 P 3550 6350
-F 0 "U4" H 3340 6540 50  0000 L CNN
-F 1 "MOC3063S-TA1" H 3550 6550 50  0000 L CNN
+F 0 "U4" H 3550 6675 50  0000 C CNN
+F 1 "MOC3063S-TA1" H 3550 6584 50  0000 C CNN
 F 2 "Devices_MSS:MOC306X" H 3350 6150 50  0001 L CIN
 F 3 "http://optoelectronics.liteon.com/upload/download/DS70-2001-026/MOC306X%20series%20201606.pdf" H 3525 6350 50  0001 L CNN

Commit message: lista por hacer
Parts:
- C4, C5, C6: value 100nF -> 1nF; footprint Capacitor_SMD:C_1206_3216Metric_Pad1.24x1.80mm_HandSolder -> Capacitor_THT:C_Rect_L13.0mm_W4.0mm_P10.00mm_FKS3_FKP3_MKS4; Campo4 GRM31CR72E104KW03L -> R60QF1100AA01K; Campo5 (none) -> 250Vac
- R10: value 100 -> 33; footprint Resistor_SMD:R_1210_3225Metric_Pad1.24x2.70mm_HandSolder -> Resistor_THT:R_Axial_DIN0207_L6.3mm_D2.5mm_P10.16mm_Horizontal; Campo4 ERA-6AEB101V -> PR01000103309JR500
- R11: footprint Resistor_SMD:R_1210_3225Metric_Pad1.24x2.70mm_HandSolder -> Resistor_THT:R_Axial_DIN0207_L6.3mm_D2.5mm_P10.16mm_Horizontal; Campo4 ERA-6AEB101V -> PR01000103309JR500
- R9: value 100 -> 33; footprint Resistor_SMD:R_1210_3225Metric_Pad1.24x2.70mm_HandSolder -> Resistor_THT:R_Axial_DIN0207_L6.3mm_D2.5mm_P10.16mm_Horizontal; Campo4 ERA-6AEB101V -> PR01000103309JR500; Campo5 (none) -> 1W
Changed lines of the file:
@@
 U 1 1 56FDDED3
 P 5550 2300
-F 0 "R9" V 5630 2300 50  0000 C CNN
-F 1 "100" V 5550 2300 50  0000 C CNN
-F 2 "Resistor_SMD:R_1210_3225Metric_Pad1.24x2.70mm_HandSolder" V 5480 2300 50  0001 C CNN
-F 3 "https://industrial.panasonic.com/cdbs/www-data/pdf/RDM0000/AOA0000C307.pdf" H 5550 2300 50  0001 C CNN
-F 4 "ERA-6AEB101V" V 5550 2300 50  0001 C CNN "Campo4"
+F 0 "R9" H 5620 2391 50  0000 L CNN
+F 1 "33" H 5620 2300 50  0000 L CNN
+F 2 "Resistor_THT:R_Axial_DIN0207_L6.3mm_D2.5mm_P10.16mm_Horizontal" V 5480 2300 50  0001 C CNN
+F 3 "http://www.vishay.com/docs/28729/pr010203.pdf" H 5550 2300 50  0001 C CNN
+F 4 "PR01000103309JR500" V 5550 2300 50  0001 C CNN "Campo4"
+F 5 "1W" H 5620 2209 50  0000 L CNN "Campo5"
 	1    5550 2300
 	1    0    0    -1
@@
 P 5550 4300
 F 0 "R10" V 5630 4300 50  0000 C CNN
-F 1 "100" V 5550 4300 50  0000 C CNN
-F 2 "Resistor_SMD:R_1210_3225Metric_Pad1.24x2.70mm_HandSolder" V 5480 4300 50  0001 C CNN
-F 3 "https://industrial.panasonic.com/cdbs/www-data/pdf/RDM0000/AOA0000C307.pdf" H 5550 4300 50  0001 C CNN
-F 4 "ERA-6AEB101V" V 5550 4300 50  0001 C CNN "Campo4"
+F 1 "33" V 5550 4300 50  0000 C CNN
+F 2 "Resistor_THT:R_Axial_DIN0207_L6.3mm_D2.5mm_P10.16mm_Horizontal" V 5480 4300 50  0001 C CNN
+F 3 "" H 5550 4300 50  0001 C CNN
+F 4 "PR01000103309JR500" V 5550 4300 50  0001 C CNN "Campo4"
 	1    5550 4300
 	1    0    0    -1
@@
 F 0 "R11" V 5630 6150 50  0000 C CNN
 F 1 "100" V 5550 6150 50  0000 C CNN
-F 2 "Resistor_SMD:R_1210_3225Metric_Pad1.24x2.70mm_HandSolder" V 5480 6150 50  0001 C CNN
-F 3 "https://industrial.panasonic.com/cdbs/www-data/pdf/RDM0000/AOA0000C307.pdf" H 5550 6150 50  0001 C CNN
-F 4 "ERA-6AEB101V" V 5550 6150 50  0001 C CNN "Campo4"
+F 2 "Resistor_THT:R_Axial_DIN0207_L6.3mm_D2.5mm_P10.16mm_Horizontal" V 5480 6150 50  0001 C CNN
+F 3 "" H 5550 6150 50  0001 C CNN
+F 4 "PR01000103309JR500" V 5550 6150 50  0001 C CNN "Campo4"
 	1    5550 6150
 	1    0    0    -1
@@
 AR Path="/56FDEE79" Ref="C6"  Part="1"
 AR Path="/56D4C343/56D4C3A8/56FDEE79" Ref="C6"  Part="1"
-F 0 "C6" H 5575 6750 50  0000 L CNN
-F 1 "100nF" H 5575 6550 50  0000 L CNN
-F 2 "Capacitor_SMD:C_1206_3216Metric_Pad1.24x1.80mm_HandSolder" H 5588 6500 50  0001 C CNN
+F 0 "C6" H 5665 6741 50  0000 L CNN
+F 1 "1nF" H 5665 6650 50  0000 L CNN
+F 2 "Capacitor_THT:C_Rect_L13.0mm_W4.0mm_P10.00mm_FKS3_FKP3_MKS4" H 5588 6500 50  0001 C CNN
 F 3 "https://search.murata.co.jp/Ceramy/image/img/A01X/G101/ENG/GRM31CR72E104KW03-01.pdf" H 5550 6650 50  0001 C CNN
-F 4 "GRM31CR72E104KW03L" H 5550 6650 50  0001 C CNN "Campo4"
+F 4 "R60QF1100AA01K" H 5550 6650 50  0001 C CNN "Campo4"
+F 5 "250Vac" H 5665 6559 50  0000 L CNN "Campo5"
 	1    5550 6650
 	1    0    0    -1
@@
 AR Path="/56FDF00C" Ref="C5"  Part="1"
 AR Path="/56D4C343/56D4C3A8/56FDF00C" Ref="C5"  Part="1"
-F 0 "C5" H 5575 4900 50  0000 L CNN
-F 1 "100nF" H 5575 4700 50  0000 L CNN
-F 2 "Capacitor_SMD:C_1206_3216Metric_Pad1.24x1.80mm_HandSolder" H 5588 4650 50  0001 C CNN
+F 0 "C5" H 5665 4891 50  0000 L CNN
+F 1 "1nF" H 5665 4800 50  0000 L CNN
+F 2 "Capacitor_THT:C_Rect_L13.0mm_W4.0mm_P10.00mm_FKS3_FKP3_MKS4" H 5588 4650 50  0001 C CNN
 F 3 "https://search.murata.co.jp/Ceramy/image/img/A01X/G101/ENG/GRM31CR72E104KW03-01.pdf" H 5550 4800 50  0001 C CNN
-F 4 "GRM31CR72E104KW03L" H 5550 4800 50  0001 C CNN "Campo4"
+F 4 "R60QF1100AA01K" H 5550 4800 50  0001 C CNN "Campo4"
+F 5 "250Vac" H 5665 4709 50  0000 L CNN "Campo5"
 	1    5550 4800
 	1    0    0    -1
@@
 AR Path="/56FDF295" Ref="C4"  Part="1"
 AR Path="/56D4C343/56D4C3A8/56FDF295" Ref="C4"  Part="1"
-F 0 "C4" H 5575 2900 50  0000 L CNN
-F 1 "100nF" H 5575 2700 50  0000 L CNN
-F 2 "Capacitor_SMD:C_1206_3216Metric_Pad1.24x1.80mm_HandSolder" H 5588 2650 50  0001 C CNN
+F 0 "C4" H 5665 2891 50  0000 L CNN
+F 1 "1nF" H 5665 2800 50  0000 L CNN
+F 2 "Capacitor_THT:C_Rect_L13.0mm_W4.0mm_P10.00mm_FKS3_FKP3_MKS4" H 5588 2650 50  0001 C CNN
 F 3 "https://search.murata.co.jp/Ceramy/image/img/A01X/G101/ENG/GRM31CR72E104KW03-01.pdf" H 5550 2800 50  0001 C CNN
-F 4 "GRM31CR72E104KW03L" H 5550 2800 50  0001 C CNN "Campo4"
+F 4 "R60QF1100AA01K" H 5550 2800 50  0001 C CNN "Campo4"
+F 5 "250Vac" H 5665 2709 50  0000 L CNN "Campo5"
 	1    5550 2800
 	1    0    0    -1
