File: Hartware_2.0.0/D21_2550.kicad_pcb (KiCad board)
At the start: 2 copper layers, 95 x 55 mm, 70 parts, among them P1 POWER I/O, P2 TA, P3 TR, P4 ISCP, Q1 FZT493TA, Q2 FZT493TA, Q3 FZT493TA, SW1 TL3301AF160QG, SW2 TL3301AF160QG, SW3 TL3301AF160QG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

Commit message: finalinzando la placa
Parts:
- removed P2: TA, Connector_PinHeader_2.54mm:PinHeader_2x01_P2.54mm_Vertical
- removed P3: TR, Connector_PinHeader_2.54mm:PinHeader_2x01_P2.54mm_Vertical
- removed TH1: Thermistor_NTC, Resistor_SMD:R_0805_2012Metric_Pad1.15x1.50mm_HandSolder
- added J1: THR, Connector_JST:JST_XH_B04B-XH-A_1x04_P2.50mm_Vertical, F.Cu at (126.2, 122.9)
- P4: moved to B.Cu
- moved R18 1.81 mm to (132.9, 129.0)
- moved R19 1.77 mm to (127.9, 129.0)
- moved RV1 1.00 mm to (156.2, 109.0)
- moved P4 0.28 mm to (113.5, 128.8), turned to 270 degrees
Connections:
- R1 pad 2: Net-(R1-Pad2) -> Vac
Routing:
- net GND: track 386.1 -> 377.5 mm, vias 44 -> 8
- net /Cerebro/Acond NTC/T_R: track 27.0 -> 30.3 mm
- net CO: track 55.9 -> 52.8 mm
- net Net-(R1-Pad2): track 2.86 -> 0.00 mm
- net VE: track 52.1 -> 50.0 mm
- net Vac: track 57.9 -> 59.9 mm
- net VDD: track 163.6 -> 161.6 mm
- net /Cerebro/Acond NTC/T_A: track 34.0 -> 35.6 mm
- net /Cerebro/Botones/S: track 51.9 -> 53.3 mm
- net /Cerebro/Botones/P: track 48.9 -> 50.2 mm
- net /Cerebro/Botones/-: track 31.5 -> 32.6 mm
- net /Cerebro/Botones/+: track 46.6 -> 47.8 mm
- net Net-(D11-Pad7): track 8.89 -> 7.85 mm
- net Net-(L1-Pad2): track 10.1 -> 9.51 mm
Other:
- board text added: "CO"
- board text added: "MCRV2.0.0-0218"
- board text added: "NAC"
- board text added: "RE"
- board text added: "VAC"
- board text added: "VE"

Commit message: colocando conector de JST de 90grados
Parts:
- J1: footprint Connector_JST:JST_XH_B04B-XH-A_1x04_P2.50mm_Vertical -> Connector_JST:JST_XH_S04B-XH-A-1_1x04_P2.50mm_Horizontal
- moved R19 8.92 mm to (124.8, 120.6)
- moved R18 8.81 mm to (130.1, 120.7)
- moved J1 6.14 mm to (127.0, 129.0)
- moved P4 4.02 mm to (109.9, 130.5)
- moved D7 2.27 mm to (104.5, 121.5)
- moved P1 2.00 mm to (186.0, 130.2)
- moved C7 1.14 mm to (107.2, 126.0)
- moved R2 0.81 mm to (102.5, 126.5)
Routing:
- net GND: track 377.5 -> 332.5 mm, vias 8 -> 7
- net VDD: track 161.6 -> 181.1 mm, vias 6 -> 7
- net VPP: track 29.7 -> 22.5 mm, vias 0 -> 1
- net PGD: track 51.2 -> 55.1 mm
- net PGC: track 55.0 -> 58.1 mm
- net CO: track 52.8 -> 55.1 mm
- net Vac: track 59.9 -> 61.9 mm
- net VE: track 50.0 -> 52.0 mm
- net /Cerebro/Botones/S: track 53.3 -> 51.6 mm
- net Net-(C7-Pad1): track 6.45 -> 7.62 mm
- net Nac: track 85.6 -> 86.4 mm
- net VDDP: track 28.0 -> 27.7 mm, vias 1 -> 2

Commit message: lista por hacer
Parts:
- removed C7: 10uf, Capacitor_SMD:CP_Elec_4x5.3
- removed D7: 1N4148X-TP, Diode_SMD:D_SOD-523
- removed HO1: MountingHole_3.2mm_M3_DIN965_Pad, MountingHole:MountingHole_3.2mm_M3_DIN965_Pad
- added JP1: pgm, Connector_PinHeader_2.54mm:PinHeader_1x02_P2.54mm_Vertical, B.Cu at (105.0, 125.5)
- C4, C5, C6: value 100nF -> 1nF; footprint Capacitor_SMD:C_1206_3216Metric_Pad1.24x1.80mm_HandSolder -> Capacitor_THT:C_Rect_L13.0mm_W4.0mm_P10.00mm_FKS3_FKP3_MKS4
- R10, R9: value 100 -> 33; footprint Resistor_SMD:R_1210_3225Metric_Pad1.24x2.70mm_HandSolder -> Resistor_THT:R_Axial_DIN0207_L6.3mm_D2.5mm_P10.16mm_Horizontal
- R11: footprint Resistor_SMD:R_1210_3225Metric_Pad1.24x2.70mm_HandSolder -> Resistor_THT:R_Axial_DIN0207_L6.3mm_D2.5mm_P10.16mm_Horizontal
- moved C6 14.1 mm to (178.0, 117.0)
- moved C5 13.8 mm to (172.0, 117.0)
- moved C4 13.0 mm to (166.0, 117.0)
- moved R11 6.89 mm to (178.0, 102.0)
- moved R2 6.88 mm to (105.0, 120.0)
- moved R10 6.34 mm to (172.0, 102.0)
- moved R9 4.04 mm to (166.0, 102.0)
Connections:
- R2 pad 2: Net-(C7-Pad1) -> VPP
Routing:
- net Nac: track 86.4 -> 120.1 mm
- net GND: track 332.5 -> 304.3 mm, vias 7 -> 6
- net VDDP: track 27.7 -> 44.4 mm
- net VDD: track 181.1 -> 189.2 mm
- net Net-(C7-Pad1): track 7.62 -> 0.00 mm
- net CO: track 55.1 -> 60.1 mm, vias 2 -> 1
- net Net-(C4-Pad1): track 2.84 -> 4.84 mm
- net Net-(C6-Pad1): track 3.07 -> 4.84 mm
- net VPP: track 22.5 -> 24.2 mm
- net Net-(C5-Pad1): track 3.22 -> 4.84 mm
- net RE: track 40.8 -> 42.2 mm, vias 2 -> 1
- net Vac: track 61.9 -> 63.0 mm
- net VE: track 52.0 -> 51.6 mm, vias 2 -> 1
