File: Hartware_omega/omega-dock-new.kicad_pcb (KiCad board)
At the start: 2 copper layers, 57.5 x 82.5 mm, 58 parts, among them J1 USB_A, J2 Conn_01x04, P1 POWER I/O, U1 USBLC6-2, U10 Z0103MN 5AA4, U11 TLA2024IRUGT, U2 OMEGA_2, U3 AP111733, U4 PBO-3-S5, U5 MOC3063S-TA1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

Commit message: agregando modelo 3d
Parts:
- J1: value USB_A -> USB_B_Micro; footprint Connector_USB:USB_A_Horizontal -> Connector_USB:USB_Micro-B_GCT_USB3076-30-A
- U1: moved to F.Cu
- moved J1 10.8 mm to (114.3, 122.7)
- moved F1 8.11 mm to (120.5, 118.8)
- moved U1 7.25 mm to (120.8, 123.5), turned to 180 degrees
Connections:
- J1 pad 4: GND -> (no net)
Routing:
- net +3V3: track 89.7 -> 22.0 mm, vias 1 -> 0
- net GND: track 288.7 -> 254.3 mm
- net +5V: track 83.3 -> 55.7 mm
- net /D+: track 10.6 -> 0.00 mm
- net /D-: track 10.6 -> 0.00 mm
- net /UD+: track 7.14 -> 0.00 mm
- net /UD-: track 6.93 -> 0.00 mm
- net Net-(F1-Pad2): track 3.00 -> 0.00 mm
