File: Hartware_omega/omega-dock-new.kicad_pcb (KiCad board)
At the start: 2 copper layers, 57.5 x 82.5 mm, 58 parts, among them J1 USB_B_Micro, J2 Conn_01x04, P1 POWER I/O, U1 USBLC6-2, U10 Z0103MN 5AA4, U11 TLA2024IRUGT, U2 OMEGA_2, U3 AP111733, U4 PBO-3-S5, U5 MOC3063S-TA1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

Commit message: culminando hartware omega 2
Parts:
- removed D4: PWR, LED_SMD:LED_0805_2012Metric_Castellated
- removed F1: 1.5A, Capacitor_SMD:C_1206_3216Metric_Pad1.24x1.80mm_HandSolder
- removed R8: 150R, Resistor_SMD:R_0805_2012Metric_Pad1.15x1.50mm_HandSolder
- removed the REF** at (164.3, 63.3)
- removed the REF** at (165.0, 135.0)
- added BT1: 3V, Battery:BatteryHolder_Keystone_3000_1x12mm, F.Cu at (134.2, 118.9)
- added D6: LED, LED_SMD:LED_0603_1608Metric_Castellated, F.Cu at (116.3, 114.5)
- added R22: 100, Resistor_SMD:R_0805_2012Metric_Pad1.29x1.40mm_HandSolder, F.Cu at (122.0, 114.5)
- added REF**: MountingHole_2.5mm_Pad_Via, MountingHole:MountingHole_2.5mm_Pad_Via, F.Cu at (116.0, 89.0)
- added REF**: MountingHole_2.5mm_Pad_Via, MountingHole:MountingHole_2.5mm_Pad_Via, F.Cu at (164.0, 63.0)
- added REF**: MountingHole_2.5mm_Pad_Via, MountingHole:MountingHole_2.5mm_Pad_Via, F.Cu at (164.0, 136.0)
- added U12: DS1307Z+, Package_SO:SOIC-8_3.9x4.9mm_P1.27mm, B.Cu at (134.0, 130.0)
- added Y1: 32.768KHZ, Crystal:Crystal_AT310_D3.0mm_L10.0mm_Horizontal, F.Cu at (147.8, 125.0)
- C1: value 10uF -> 22uF
- C9: footprint Capacitor_SMD:CP_Elec_6.3x5.3 -> Capacitor_SMD:CP_Elec_4x5.3
- D1, D2, D3: footprint LED_SMD:LED_0805_2012Metric_Castellated -> LED_SMD:LED_0603_1608Metric_Castellated
- D5: value D -> Bridge; footprint Diode_SMD:D_0805_2012Metric_Pad0.97x1.50mm_HandSolder -> Devices_MSS:MBS -1
- J1: footprint Connector_USB:USB_Micro-B_GCT_USB3076-30-A -> Devices_MSS:USB_Micro-B_10118193-0001LF
- R1, R2, R3: value 220 -> 100
- R19: value 43.5K -> 604K; footprint Resistor_SMD:R_0805_2012Metric_Pad1.15x1.50mm_HandSolder -> Resistor_SMD:R_0805_2012Metric_Pad1.29x1.40mm_HandSolder
- R20: value 1K -> 604K; footprint Resistor_SMD:R_0805_2012Metric_Pad1.15x1.50mm_HandSolder -> Resistor_SMD:R_0805_2012Metric_Pad1.29x1.40mm_HandSolder
- R21: value 43.5K -> 10k; footprint Resistor_SMD:R_0805_2012Metric_Pad1.15x1.50mm_HandSolder -> Resistor_SMD:R_0805_2012Metric_Pad1.29x1.40mm_HandSolder
- R4, R5: value 10K -> 2.2K
- U1: moved to B.Cu
- moved R20 12.1 mm to (129.5, 104.5)
- moved R19 8.12 mm to (125.0, 104.5)
- moved D5 4.48 mm to (125.5, 97.5), turned to 90 degrees
- moved R1 4.00 mm to (120.0, 101.0)
- moved R3 4.00 mm to (120.0, 93.0)
- moved R2 3.96 mm to (120.0, 97.0)
- moved D1 3.00 mm to (116.0, 101.0)
- moved D3 3.00 mm to (116.0, 93.0)
- moved R21 2.92 mm to (136.5, 99.5)
- moved D2 2.88 mm to (116.0, 97.0)
- moved C1 2.82 mm to (136.5, 104.0)
- moved C12 2.50 mm to (160.0, 108.5)
- moved C9 2.50 mm to (162.5, 109.0)
- moved C11 2.00 mm to (162.0, 102.0)
- moved U1 1.15 mm to (121.9, 123.7), turned to 0 degrees
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Connections:
- D5 pad 2: Vac -> GND
- J1 pad 1: Net-(F1-Pad2) -> +5V
- R19 pad 1: Net-(R19-Pad1) -> Net-(D5-Pad1)
- R19 pad 2: /V_TEST -> Net-(R19-Pad2)
- R20 pad 1: /V_TEST -> Net-(R19-Pad2)
- R20 pad 2: GND -> /V_TEST
- R21 pad 1: Net-(D5-Pad1) -> /V_TEST
- R21 pad 2: Net-(R19-Pad1) -> GND
- U1 pad 5: +3V3 -> +5V
- U2 pad 2: (no net) -> /error
Routing:
- net +5V: track 55.7 -> 114.3 mm, vias 1 -> 2
- net GND: track 254.3 -> 305.8 mm, vias 2 -> 1
- net +3V3: track 22.0 -> 72.9 mm, vias 0 -> 1
- net +BATT: track 0.00 -> 40.4 mm, vias 0 -> 1
- net /SCL: track 14.8 -> 38.0 mm, vias 0 -> 1
- net /SDA: track 14.7 -> 32.6 mm, vias 0 -> 1
- net /D-: track 0.00 -> 13.9 mm
- net Net-(U12-Pad1): track 0.00 -> 13.3 mm
- net /D+: track 0.00 -> 12.2 mm
- net Net-(U12-Pad2): track 0.00 -> 10.4 mm
- net Nac: track 94.4 -> 101.9 mm
- net Net-(R19-Pad1): track 5.68 -> 0.00 mm
- net /UD+: track 0.00 -> 5.28 mm, vias 0 -> 1
- net /UD-: track 0.00 -> 4.76 mm, vias 0 -> 1
- net /error: track 0.00 -> 4.50 mm
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- added copper zone on B.Cu, net GND
- added copper zone on F.Cu, net GND

Commit message: pasandome a mac
Parts:
- removed R9: 300k, Resistor_SMD:R_1206_3216Metric_Pad1.24x1.80mm_HandSolder
- removed U1: USBLC6-2, Package_TO_SOT_SMD:SOT-23-6_Handsoldering
- added D4: LED, LED_SMD:LED_0603_1608Metric_Castellated, F.Cu at (114.3, 108.5)
- added D7: LED, LED_SMD:LED_0603_1608Metric_Castellated, F.Cu at (114.3, 111.6)
- added F1: 1A, Devices_MSS:FC-211-22_M, B.Cu at (164.5, 73.0)
- added GPIO: TestPoint_Pad_D1.5mm, TestPoint:TestPoint_Pad_D1.5mm, F.Cu at (147.0, 137.5)
- added R23: 10K, Resistor_SMD:R_0805_2012Metric_Pad1.29x1.40mm_HandSolder, F.Cu at (117.0, 131.0)
- added R24: 100, Resistor_SMD:R_0805_2012Metric_Pad1.29x1.40mm_HandSolder, F.Cu at (117.3, 114.1)
- added R8: 100, Resistor_SMD:R_0805_2012Metric_Pad1.29x1.40mm_HandSolder, F.Cu at (118.0, 109.5)
- added SW1: RST, Button_Switch_SMD:Panasonic_EVQPUL_EVQPUC, F.Cu at (115.0, 124.4)
- added VT: TestPoint_Pad_D1.5mm, TestPoint:TestPoint_Pad_D1.5mm, F.Cu at (131.5, 107.1)
- J1: value USB_B_Micro -> SI; footprint Devices_MSS:USB_Micro-B_10118193-0001LF -> Devices_MSS:HE_XDF1B_1x03_P2.50mm_Horizontal
- J2: value Conn_01x04 -> Termistor; moved to F.Cu
- P1: footprint TerminalBlock:TerminalBlock_bornier-5_P5.08mm -> Devices_MSS:WE-3221 - 3.50MM
- moved J1 49.0 mm to (162.5, 133.0), turned to 90 degrees
- moved REF** 30.5 mm to (133.5, 62.0)
- moved P1 17.3 mm to (154.2, 63.2), turned to 180 degrees
- moved R22 9.23 mm to (120.0, 105.5)
- moved D6 9.23 mm to (114.3, 105.5)
- moved REF** 8.14 mm to (156.0, 137.5)
- moved R6 5.84 mm to (156.5, 118.0)
- moved J2 5.03 mm to (164.0, 123.0), turned to 90 degrees
- moved R7 4.96 mm to (156.5, 123.0)
- moved D3 3.89 mm to (114.3, 96.5)
- moved R3 3.50 mm to (120.0, 96.5)
- moved D2 3.02 mm to (114.3, 99.5)
- moved R2 2.50 mm to (120.0, 99.5)
- moved D1 2.27 mm to (114.3, 102.5)
- moved R1 1.50 mm to (120.0, 102.5)
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Connections:
- D5 pad 1: Net-(D5-Pad1) -> VacF
- D5 pad 2: GND -> Nac
- D5 pad 3: Vac -> Net-(D5-Pad3)
- D5 pad 4: Nac -> GND
- J1 pad 2: /UD- -> /I_TEST
- J1 pad 3: /UD+ -> GND
- L2 pad 1: Net-(L2-Pad1) -> VacF
- P1 pad 1: Vac -> Nac
- P1 pad 2: CO -> VE
- P1 pad 4: VE -> CO
- P1 pad 5: Nac -> Vac
- R19 pad 1: Net-(D5-Pad1) -> Net-(D5-Pad3)
- R6 pad 1: +5V -> +3V3
- R7 pad 1: +5V -> +3V3
- RV1 pad 1: Vac -> VacF
- U11 pad 4: Net-(J2-Pad3) -> Net-(J2-Pad1)
- U11 pad 5: Net-(J2-Pad1) -> Net-(J2-Pad3)
- U11 pad 7: (no net) -> /I_TEST
- U11 pad 8: +5V -> +3V3
- U2 pad 19: (no net) -> /GPIO
- U2 pad 20: (no net) -> /red
- U2 pad 26: (no net) -> Net-(R23-Pad1)
- U2 pad 29: /D- -> (no net)
- U2 pad 30: /D+ -> (no net)
Routing:
- net GND: track 305.8 -> 71.3 mm, vias 1 -> 0
- net VacF: track 0.00 -> 60.0 mm
- net /GPIO: track 0.00 -> 53.3 mm, vias 0 -> 1
- net /red: track 0.00 -> 48.1 mm, vias 0 -> 1
- net +3V3: track 72.9 -> 116.3 mm
- net Net-(R23-Pad1): track 0.00 -> 31.7 mm
- net Nac: track 101.9 -> 78.5 mm
- net /I_TEST: track 0.00 -> 17.3 mm, vias 0 -> 1
- net /D-: track 13.9 -> 0.00 mm
- net /D+: track 12.2 -> 0.00 mm
- net Vac: track 45.6 -> 33.8 mm
- net /V_TEST: track 43.9 -> 52.6 mm
- net Net-(L2-Pad1): track 5.83 -> 0.00 mm
- net /SCL: track 38.0 -> 32.3 mm, vias 1 -> 2
- net /UD+: track 5.28 -> 0.00 mm, vias 1 -> 0
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Other:
- outline, holes or cut-outs redrawn
- board text added: "RST"
- board text added: "SCR0418V1.0.0"
