File: Hartware_omega/FuenteST.sch (KiCad schematic (older format))
At the start: 14 parts, among them U3 AP111733, U4 PBO-3-S5

Commit message: culminando hartware omega 2
Parts:
- C10: Campo4 EEE-FKC271XSP -> EEE-FK0J271SP
- C12: Campo4 C1206C104K5RAC7867 -> C1206X104J3JACAUTO
- C7: Campo4 (none) -> EEE-1VA100SR
- C9: footprint Capacitor_SMD:CP_Elec_6.3x5.3 -> Capacitor_SMD:CP_Elec_4x5.3; Campo4 (none) -> EEE-1AA101WR
- R9: Campo4 (none) -> RC1206FR-07300KL
- U3: Campo4 (none) -> TLV1117-33CDCYR
Changed lines of the file:
@@
 F 2 "Resistor_SMD:R_1206_3216Metric_Pad1.24x1.80mm_HandSolder" V 4530 3650 30  0001 C CNN
 F 3 "" H 4600 3650 30  0000 C CNN
+F 4 "RC1206FR-07300KL" V 4600 3650 50  0001 C CNN "Campo4"
 	1    4600 3650
 	0    1    1    0
@@
 F 2 "Capacitor_SMD:CP_Elec_6.3x7.7" H 7250 3850 50  0001 C CNN
 F 3 "https://media.digikey.com/pdf/Data%20Sheets/Panasonic%20Capacitors%20PDFs/FKS_Series_Type_V.pdf" H 7250 3850 50  0001 C CNN
-F 4 "EEE-FKC271XSP" H 7250 3850 50  0001 C CNN "Campo4"
+F 4 "EEE-FK0J271SP" H 7250 3850 50  0001 C CNN "Campo4"
 	1    7250 3850
 	1    0    0    -1
@@
 F 1 "100nF" H 8315 3805 50  0000 L CNN
 F 2 "Capacitor_SMD:C_1206_3216Metric_Pad1.24x1.80mm_HandSolder" H 8238 3700 50  0001 C CNN
-F 3 "https://search.kemet.com/component-edge/download/datasheet/C1206C104K5RACTU.pdf" H 8200 3850 50  0001 C CNN
-F 4 "C1206C104K5RAC7867" H 8200 3850 50  0001 C CNN "Campo4"
+F 3 "" H 8200 3850 50  0001 C CNN
+F 4 "C1206X104J3JACAUTO" H 8200 3850 50  0001 C CNN "Campo4"
 	1    8200 3850
 	1    0    0    -1
@@
 F 0 "C9" H 7015 2746 50  0000 L CNN
 F 1 "100uF" H 7015 2655 50  0000 L CNN
-F 2 "Capacitor_SMD:CP_Elec_6.3x5.3" H 6900 2700 50  0001 C CNN
+F 2 "Capacitor_SMD:CP_Elec_4x5.3" H 6900 2700 50  0001 C CNN
 F 3 "" H 6900 2700 50  0001 C CNN
+F 4 "EEE-1AA101WR" H 6900 2700 50  0001 C CNN "Campo4"
 	1    6900 2700
 	1    0    0    -1
@@
 F 2 "Capacitor_SMD:CP_Elec_4x5.3" H 5850 2700 50  0001 C CNN
 F 3 "" H 5850 2700 50  0001 C CNN
+F 4 "EEE-1VA100SR" H 5850 2700 50  0001 C CNN "Campo4"
 	1    5850 2700
 	1    0    0    -1
@@
 F 2 "Package_TO_SOT_SMD:SOT-223" H 6450 2150 50  0001 C CNN
 F 3 "" H 6550 2250 50  0001 C CNN
+F 4 "TLV1117-33CDCYR" H 6450 2500 50  0001 C CNN "Campo4"
 	1    6450 2500
 	1    0    0    -1

Commit message: pasandome a mac
Parts:
- removed R9: 300k, Resistor_SMD:R_1206_3216Metric_Pad1.24x1.80mm_HandSolder, symbol Device:R
- added F1: 1A, Devices_MSS:FC-211-22_M, symbol Device:Fuse
- C12: Campo4 C1206X104J3JACAUTO -> GCM21BR72A104KA37L
- U3: symbol omega-dock-new-rescue:AP111733-RESCUE-omega-dock-new -> Regulator_Linear:AP1117-33
Connections:
- net labels added: VacF
- wire segments 45 -> 51
Other:
- moved on the sheet: C9, RV1
Changed lines of the file:
@@
 Comment4 ""
 $EndDescr
-Text GLabel 3650 4250 0    60   Input ~ 0
+Text GLabel 4000 4250 0    60   Input ~ 0
 Nac
-Text GLabel 3650 3650 0    60   Input ~ 0
+Text GLabel 4000 3650 0    60   Input ~ 0
 Vac
 $Comp
@@
 $EndComp
 $Comp
-L Device:R R9
-U 1 1 56F82842
-P 4600 3650
-F 0 "R9" V 4680 3650 40  0000 C CNN
-F 1 "300k" V 4607 3651 40  0000 C CNN
-F 2 "Resistor_SMD:R_1206_3216Metric_Pad1.24x1.80mm_HandSolder" V 4530 3650 30  0001 C CNN
-F 3 "" H 4600 3650 30  0000 C CNN
-F 4 "RC1206FR-07300KL" V 4600 3650 50  0001 C CNN "Campo4"
-	1    4600 3650
-	0    1    1    0
-$EndComp
-$Comp
 L Mss_devices:PBO-3-S5 U4
 U 1 1 5A7C683A
@@
 	5750 4050 5750 4250
 Wire Wire Line
-	5750 4250 4200 4250
+	5750 4250 4650 4250
 $Comp
 L Device:L_Core_Ferrite L2
@@
 	5550 3650 5850 3650
 Wire Wire Line
-	5250 3650 4750 3650
+	5250 3650 4950 3650
 $Comp
 L Device:Varistor RV1
 U 1 1 5A7D0BB3
-P 4200 3950
-F 0 "RV1" H 3900 4000 50  0000 L CNN
-F 1 "B72214S0351K101" H 3350 3900 50  0000 L CNN
-F 2 "Capacitor_THT:C_Disc_D4.3mm_W1.9mm_P5.00mm" V 4130 3950 50  0001 C CNN
-F 3 "https://en.tdk.eu/inf/70/db/var_11/SIOV_Leaded_StandarD.pdf" H 4200 3950 50  0001 C CNN
-F 4 "B72214S0351K101" H 4200 3950 50  0001 C CNN "Campo4"
-	1    4200 3950
-	1    0    0    -1
-$EndComp
-Wire Wire Line
-	4200 3800 4200 3650
-Wire Wire Line
-	4200 4100 4200 4250
-Connection ~ 4200 4250
-Wire Wire Line
-	4200 4250 3650 4250
-Wire Wire Line
-	3650 3650 4200 3650
-Connection ~ 4200 3650
+P 4650 3950
+F 0 "RV1" H 4350 4000 50  0000 L CNN
+F 1 "B72214S0351K101" H 3800 3900 50  0000 L CNN
+F 2 "Capacitor_THT:C_Disc_D4.3mm_W1.9mm_P5.00mm" V 4580 3950 50  0001 C CNN
+F 3 "https://en.tdk.eu/inf/70/db/var_11/SIOV_Leaded_StandarD.pdf" H 4650 3950 50  0001 C CNN
+F 4 "B72214S0351K101" H 4650 3950 50  0001 C CNN "Campo4"
+	1    4650 3950
+	1    0    0    -1
+$EndComp
+Wire Wire Line
+	4650 3800 4650 3650
+Wire Wire Line
+	4650 4100 4650 4250
+Connection ~ 4650 4250
+Wire Wire Line
+	4650 4250 4000 4250
 $Comp
 L Device:C C8
@@
 F 2 "Capacitor_SMD:C_1206_3216Metric_Pad1.24x1.80mm_HandSolder" H 8238 3700 50  0001 C CNN
 F 3 "" H 8200 3850 50  0001 C CNN
-F 4 "C1206X104J3JACAUTO" H 8200 3850 50  0001 C CNN "Campo4"
+F 4 "GCM21BR72A104KA37L" H 8200 3850 50  0001 C CNN "Campo4"
 	1    8200 3850
 	1    0    0    -1
@@
 Wire Wire Line
 	8200 4050 7750 4050
-Wire Wire Line
-	4200 3650 4450 3650
 $Comp
 L power:+3.3V #PWR018
 U 1 1 5AA1AACA
-P 6900 2400
-F 0 "#PWR018" H 6900 2250 50  0001 C CNN
-F 1 "+3.3V" H 6900 2540 50  0000 C CNN
-F 2 "" H 6900 2400 50  0001 C CNN
-F 3 "" H 6900 2400 50  0001 C CNN
-	1    6900 2400
+P 7000 2400
+F 0 "#PWR018" H 7000 2250 50  0001 C CNN
+F 1 "+3.3V" H 7000 2540 50  0000 C CNN
+F 2 "" H 7000 2400 50  0001 C CNN
+F 3 "" H 7000 2400 50  0001 C CNN
+	1    7000 2400
 	1    0    0    -1
 $EndComp
@@
 L power:GND #PWR017
 U 1 1 5AA1AADA
-P 6450 2800
-F 0 "#PWR017" H 6450 2550 50  0001 C CNN
-F 1 "GND" H 6450 2650 50  0000 C CNN
-F 2 "" H 6450 2800 50  0001 C CNN
-F 3 "" H 6450 2800 50  0001 C CNN
-	1    6450 2800
+P 6450 2900
+F 0 "#PWR017" H 6450 2650 50  0001 C CNN
+F 1 "GND" H 6450 2750 50  0000 C CNN
+F 2 "" H 6450 2900 50  0001 C CNN
+F 3 "" H 6450 2900 50  0001 C CNN
+	1    6450 2900
 	1    0    0    -1
 $EndComp
@@
 L power:GND #PWR019
 U 1 1 5AA1AAE0
-P 6900 2900
-F 0 "#PWR019" H 6900 2650 50  0001 C CNN
-F 1 "GND" H 6900 2750 50  0000 C CNN
-F 2 "" H 6900 2900 50  0001 C CNN
-F 3 "" H 6900 2900 50  0001 C CNN
-	1    6900 2900
-	1    0    0    -1
-$EndComp
-Wire Wire Line
-	6900 2500 6900 2550
-Wire Wire Line
-	6900 2400 6900 2500
-Connection ~ 6900 2500
-Wire Wire Line
-	6750 2500 6900 2500
+P 7000 2900
+F 0 "#PWR019" H 7000 2650 50  0001 C CNN
+F 1 "GND" H 7000 2750 50  0000 C CNN
+F 2 "" H 7000 2900 50  0001 C CNN
+F 3 "" H 7000 2900 50  0001 C CNN
+	1    7000 2900
+	1    0    0    -1
+$EndComp
+Wire Wire Line
+	7000 2500 7000 2550
+Wire Wire Line
+	7000 2400 7000 2500
+Connection ~ 7000 2500
+Wire Wire Line
+	6750 2500 6800 2500
 $Comp
 L Device:CP1 C9
 U 1 1 5AA1AAEA
-P 6900 2700
-F 0 "C9" H 7015 2746 50  0000 L CNN
-F 1 "100uF" H 7015 2655 50  0000 L CNN
-F 2 "Capacitor_SMD:CP_Elec_4x5.3" H 6900 2700 50  0001 C CNN
-F 3 "" H 6900 2700 50  0001 C CNN
-F 4 "EEE-1AA101WR" H 6900 2700 50  0001 C CNN "Campo4"
-	1    6900 2700
+P 7000 2700
+F 0 "C9" H 7115 2746 50  0000 L CNN
+F 1 "100uF" H 7115 2655 50  0000 L CNN
+F 2 "Capacitor_SMD:CP_Elec_4x5.3" H 7000 2700 50  0001 C CNN
+F 3 "" H 7000 2700 50  0001 C CNN
+F 4 "EEE-1AA101WR" H 7000 2700 50  0001 C CNN "Campo4"
+	1    7000 2700
 	1    0    0    -1
 $EndComp
@@
 $EndComp
 $Comp
-L omega-dock-new-rescue:AP111733-RESCUE-omega-dock-new U3
+L Regulator_Linear:AP1117-33 U3
 U 1 1 5AA1AAF8
 P 6450 2500
 F 0 "U3" H 6550 2250 50  0000 C CNN
-F 1 "AP111733" H 6450 2750 50  0000 C CNN
+F 1 "AP111733" H 6450 2650 50  0000 C CNN
 F 2 "Package_TO_SOT_SMD:SOT-223" H 6450 2150 50  0001 C CNN
 F 3 "" H 6550 2250 50  0001 C CNN
@@
 	5850 2900 5850 2850
 Wire Wire Line
-	6900 2900 6900 2850
+	7000 2900 7000 2850
+Wire Wire Line
+	6450 2900 6450 2800
+$Comp
+L Device:Fuse F1
+U 1 1 5B12EF1D
+P 4300 3650
+F 0 "F1" V 4103 3650 50  0000 C CNN
+F 1 "1A" V 4194 3650 50  0000 C CNN
+F 2 "Devices_MSS:FC-211-22_M" V 4230 3650 50  0001 C CNN
+F 3 "~" H 4300 3650 50  0001 C CNN
+F 4 "FC-211-22" V 4300 3650 50  0001 C CNN "Campo4"
+	1    4300 3650
+	0    1    1    0
+$EndComp
+Text GLabel 4950 3550 1    60   Output ~ 0
+VacF
+Wire Wire Line
+	4950 3550 4950 3650
+Connection ~ 4950 3650
+Wire Wire Line
+	4450 3650 4650 3650
+Connection ~ 4650 3650
+Wire Wire Line
+	4150 3650 4000 3650
+Wire Wire Line
+	4650 3650 4950 3650
+Wire Wire Line
+	6750 2650 6800 2650
+Wire Wire Line
+	6800 2650 6800 2500
+Connection ~ 6800 2500
+Wire Wire Line
+	6800 2500 7000 2500
 $EndSCHEMATC
