File: Hartware_omega/OutTriac.sch (KiCad schematic (older format))
At the start: 19 parts, among them P1 POWER I/O, U10 Z0103MN 5AA4, U5 MOC3063S-TA1, U6 MOC3063S-TA1, U7 MOC3063S-TA1, U8 Z0103MN 5AA4, U9 Z0103MN 5AA4

Commit message: culminando hartware omega 2
Parts:
- R10, R11, R12, R13, R14, R15: Campo4 ESR10EZPJ331 -> RCS0805330RFKEA
Changed lines of the file:
@@
 F 2 "Resistor_SMD:R_0805_2012Metric_Pad1.15x1.50mm_HandSolder" V 3080 2350 50  0001 C CNN
 F 3 "http://www.rohm.com/web/global/datasheet/ESR01MZPF/esr-e" H 3150 2350 50  0001 C CNN
-F 4 "ESR10EZPJ331" V 3150 2350 50  0001 C CNN "Campo4"
+F 4 "RCS0805330RFKEA" V 3150 2350 50  0001 C CNN "Campo4"
 	1    3150 2350
 	1    0    0    -1
@@
 F 2 "Resistor_SMD:R_0805_2012Metric_Pad1.15x1.50mm_HandSolder" V 4330 1400 50  0001 C CNN
 F 3 "http://www.rohm.com/web/global/datasheet/ESR01MZPF/esr-e" H 4400 1400 50  0001 C CNN
-F 4 "ESR10EZPJ331" V 4400 1400 50  0001 C CNN "Campo4"
+F 4 "RCS0805330RFKEA" V 4400 1400 50  0001 C CNN "Campo4"
 	1    4400 1400
 	0    1    1    0
@@
 F 2 "Resistor_SMD:R_0805_2012Metric_Pad1.15x1.50mm_HandSolder" V 4280 3500 50  0001 C CNN
 F 3 "http://www.rohm.com/web/global/datasheet/ESR01MZPF/esr-e" H 4350 3500 50  0001 C CNN
-F 4 "ESR10EZPJ331" V 4350 3500 50  0001 C CNN "Campo4"
+F 4 "RCS0805330RFKEA" V 4350 3500 50  0001 C CNN "Campo4"
 	1    4350 3500
 	0    1    1    0
@@
 F 2 "Resistor_SMD:R_0805_2012Metric_Pad1.15x1.50mm_HandSolder" V 3030 4450 50  0001 C CNN
 F 3 "http://www.rohm.com/web/global/datasheet/ESR01MZPF/esr-e" H 3100 4450 50  0001 C CNN
-F 4 "ESR10EZPJ331" V 3100 4450 50  0001 C CNN "Campo4"
+F 4 "RCS0805330RFKEA" V 3100 4450 50  0001 C CNN "Campo4"
 	1    3100 4450
 	1    0    0    -1
@@
 F 2 "Resistor_SMD:R_0805_2012Metric_Pad1.15x1.50mm_HandSolder" V 4280 5600 50  0001 C CNN
 F 3 "http://www.rohm.com/web/global/datasheet/ESR01MZPF/esr-e" H 4350 5600 50  0001 C CNN
-F 4 "ESR10EZPJ331" V 4350 5600 50  0001 C CNN "Campo4"
+F 4 "RCS0805330RFKEA" V 4350 5600 50  0001 C CNN "Campo4"
 	1    4350 5600
 	0    1    1    0
@@
 F 2 "Resistor_SMD:R_0805_2012Metric_Pad1.15x1.50mm_HandSolder" V 3030 6550 50  0001 C CNN
 F 3 "http://www.rohm.com/web/global/datasheet/ESR01MZPF/esr-e" H 3100 6550 50  0001 C CNN
-F 4 "ESR10EZPJ331" V 3100 6550 50  0001 C CNN "Campo4"
+F 4 "RCS0805330RFKEA" V 3100 6550 50  0001 C CNN "Campo4"
 	1    3100 6550
 	1    0    0    -1

Commit message: pasandome a mac
Parts:
- P1: footprint TerminalBlock:TerminalBlock_bornier-5_P5.08mm -> Devices_MSS:WE-3221 - 3.50MM; Campo4 282836-5 -> 691322110005
Connections:
- net CO: now also P1.4 (Pin_4); no longer P1.2 (Pin_2)
- net Nac: now also P1.1 (Pin_1); no longer P1.5 (Pin_5)
- net VE: now also P1.2 (Pin_2); no longer P1.4 (Pin_4)
- net Vac: now also P1.5 (Pin_5); no longer P1.1 (Pin_1)
Changed lines of the file:
@@
 F 0 "P1" H 8250 4550 50  0000 C CNN
 F 1 "POWER I/O" V 8350 4200 50  0000 C CNN
-F 2 "TerminalBlock:TerminalBlock_bornier-5_P5.08mm" H 8250 4200 50  0001 C CNN
-F 3 "http://www.te.com/commerce/DocumentDelivery/DDEController?Action=srchrtrv&DocNm=282836&DocType=Customer+Drawing&DocLang=English" H 8250 4200 50  0001 C CNN
-F 4 "282836-5" H 8250 4200 50  0001 C CNN "Campo4"
+F 2 "Devices_MSS:WE-3221 - 3.50MM" H 8250 4200 50  0001 C CNN
+F 3 "http://katalog.we-online.de/em/datasheet/6913221100xx.pdf" H 8250 4200 50  0001 C CNN
+F 4 "691322110005" H 8250 4200 50  0001 C CNN "Campo4"
 	1    8250 4200
-	1    0    0    -1
+	1    0    0    1
 $EndComp
 Wire Wire Line
