File: Hartware_omega/omega-dock-new.sch (KiCad schematic (older format))
At the start: 23 parts, among them J1 USB_A, J2 Conn_01x04, U1 USBLC6-2, U11 TLA2024IRUGT, U2 OMEGA_2

Commit message: agregando modelo 3d
Parts:
- removed J1: USB_A, Connector_USB:USB_A_Horizontal, symbol omega-dock-new-rescue:USB_A-RESCUE-omega-dock-new
- added J1: USB_B_Micro, Connector_USB:USB_Micro-B_GCT_USB3076-30-A, symbol Connector_Specialized:USB_B_Micro
Connections:
- net GND: now also J1.5 (GND), J1.6 (Shield)
- net UD+: now also J1.3 (D+)
- net UD-: now also J1.2 (D-)
- net at F1.2: now also J1.1 (VBUS)
Other:
- moved on the sheet: R7
Changed lines of the file:
@@
 $EndDescr
 $Comp
-L omega-dock-new-rescue:USB_A-RESCUE-omega-dock-new J1
-U 1 1 5950B98B
-P 1450 1950
-F 0 "J1" H 1250 2400 50  0000 L CNN
-F 1 "USB_A" H 1250 2300 50  0000 L CNN
-F 2 "Connector_USB:USB_A_Horizontal" H 1600 1900 50  0001 C CNN
-F 3 "" H 1600 1900 50  0001 C CNN
-	1    1450 1950
-	1    0    0    -1
-$EndComp
-$Comp
-L power1:+5V #PWR02
+L power:+5V #PWR02
 U 1 1 5950BD7E
 P 1800 1450
@@
 	1950 2100 2600 2100
 $Comp
-L power1:GND #PWR03
+L power:GND #PWR03
 U 1 1 595105A0
 P 2400 2150
@@
 $EndComp
 $Comp
-L power1:+3.3V #PWR05
+L power:+3.3V #PWR05
 U 1 1 59510668
 P 3650 1650
@@
 	5700 3650 5500 3650
 $Comp
-L power1:GND #PWR01
+L power:GND #PWR01
 U 1 1 59512193
 P 1450 2500
@@
 	5500 2950 5500 3350
 $Comp
-L power1:GND #PWR06
+L power:GND #PWR06
 U 1 1 595130B7
 P 3700 3200
@@
 $EndComp
 $Comp
-L power1:+3.3V #PWR08
+L power:+3.3V #PWR08
 U 1 1 595130E9
 P 5700 3400
@@
 $EndComp
 $Comp
-L power1:+3.3V #PWR010
+L power:+3.3V #PWR010
 U 1 1 598696ED
 P 6850 3000
@@
 $EndComp
 $Comp
-L power1:GND #PWR011
+L power:GND #PWR011
 U 1 1 5986977F
 P 6850 3600
@@
 L Device:R R7
 U 1 1 5AD3D220
-P 8950 5350
-F 0 "R7" H 9020 5396 50  0000 L CNN
-F 1 "10K" H 9020 5305 50  0000 L CNN
-F 2 "Resistor_SMD:R_0805_2012Metric_Pad1.15x1.50mm_HandSolder" V 8880 5350 50  0001 C CNN
-F 3 "~" H 8950 5350 50  0001 C CNN
-	1    8950 5350
+P 8750 5350
+F 0 "R7" H 8820 5396 50  0000 L CNN
+F 1 "10K" H 8820 5305 50  0000 L CNN
+F 2 "Resistor_SMD:R_0805_2012Metric_Pad1.15x1.50mm_HandSolder" V 8680 5350 50  0001 C CNN
+F 3 "~" H 8750 5350 50  0001 C CNN
+	1    8750 5350
 	1    0    0    -1
 $EndComp
@@
 	8450 5650 8450 5500
 Wire Wire Line
-	8950 5500 8950 5550
-Wire Wire Line
-	7700 5550 8950 5550
+	8750 5500 8750 5550
+Wire Wire Line
+	7700 5550 8750 5550
 $Comp
 L power:GND #PWR013
@@
 	8450 5200 8450 5100
 Wire Wire Line
-	8450 5100 8700 5100
-Wire Wire Line
-	8950 5100 8950 5200
+	8450 5100 8600 5100
+Wire Wire Line
+	8750 5100 8750 5200
 $Comp
 L power:+5V #PWR09
@@
 L power:+5V #PWR012
 U 1 1 5AD4BDDB
-P 8700 5050
-F 0 "#PWR012" H 8700 4900 50  0001 C CNN
-F 1 "+5V" H 8715 5223 50  0000 C CNN
-F 2 "" H 8700 5050 50  0001 C CNN
-F 3 "" H 8700 5050 50  0001 C CNN
-	1    8700 5050
-	1    0    0    -1
-$EndComp
-Wire Wire Line
-	8700 5050 8700 5100
-Connection ~ 8700 5100
-Wire Wire Line
-	8700 5100 8950 5100
+P 8600 5050
+F 0 "#PWR012" H 8600 4900 50  0001 C CNN
+F 1 "+5V" H 8615 5223 50  0000 C CNN
+F 2 "" H 8600 5050 50  0001 C CNN
+F 3 "" H 8600 5050 50  0001 C CNN
+	1    8600 5050
+	1    0    0    -1
+$EndComp
+Wire Wire Line
+	8600 5050 8600 5100
+Connection ~ 8600 5100
+Wire Wire Line
+	8600 5100 8750 5100
 Wire Wire Line
 	7700 5450 8050 5450
@@
 $EndComp
 Wire Wire Line
-	9200 5550 8950 5550
-Connection ~ 8950 5550
+	9200 5550 8750 5550
+Connection ~ 8750 5550
 Wire Wire Line
 	9200 5750 8450 5750
@@
 Wire Wire Line
 	10350 4100 10350 4050
+$Comp
+L Connector_Specialized:USB_B_Micro J1
+U 1 1 5AD32A50
+P 1450 1950
+F 0 "J1" H 1505 2417 50  0000 C CNN
+F 1 "USB_B_Micro" H 1505 2326 50  0000 C CNN
+F 2 "Connector_USB:USB_Micro-B_GCT_USB3076-30-A" H 1600 1900 50  0001 C CNN
+F 3 "~" H 1600 1900 50  0001 C CNN
+	1    1450 1950
+	1    0    0    -1
+$EndComp
 $EndSCHEMATC

Commit message: culminando hartware omega 2
Parts:
- removed D4: PWR, LED_SMD:LED_0805_2012Metric_Castellated, symbol Device:LED_ALT
- removed D5: D, Diode_SMD:D_0805_2012Metric_Pad0.97x1.50mm_HandSolder, symbol Device:D
- removed F1: 1.5A, Capacitor_SMD:C_1206_3216Metric_Pad1.24x1.80mm_HandSolder, symbol omega-dock-new-rescue:Polyfuse-RESCUE-omega-dock-new
- removed R8: 150R, Resistor_SMD:R_0805_2012Metric_Pad1.15x1.50mm_HandSolder, symbol Device:R
- added BT1: 3V, Battery:BatteryHolder_Keystone_3000_1x12mm, symbol Device:Battery_Cell
- added D5: Bridge, Devices_MSS:MBS -1, symbol Device:D_Bridge_+-AA
- added D6: LED, LED_SMD:LED_0603_1608Metric_Castellated, symbol Device:LED
- added R22: 100, Resistor_SMD:R_0805_2012Metric_Pad1.29x1.40mm_HandSolder, symbol Device:R
- added U12: DS1307Z+, Package_SO:SOIC-8_3.9x4.9mm_P1.27mm, symbol Timer_RTC:DS1307Z+
- added Y1: 32.768KHZ, Crystal:Crystal_AT310_D3.0mm_L10.0mm_Horizontal, symbol Device:Crystal
- C1: value 10uF -> 22uF; Campo4 (none) -> EEE-HA1V220WR
- D1, D2, D3: footprint LED_SMD:LED_0805_2012Metric_Castellated -> LED_SMD:LED_0603_1608Metric_Castellated; Campo4 (none) -> VLMB1300-GS08
- J1: footprint Connector_USB:USB_Micro-B_GCT_USB3076-30-A -> Devices_MSS:USB_Micro-B_10118193-0001LF; Campo4 (none) -> 10118193-0001LF
- J2: Campo4 (none) -> S4B-XH-A(LF)(SN)
- R1, R2, R3: value 220 -> 100; Campo4 (none) -> ERA-6AEB101V
- R19: value 43.5K -> 604K; footprint Resistor_SMD:R_0805_2012Metric_Pad1.15x1.50mm_HandSolder -> Resistor_SMD:R_0805_2012Metric_Pad1.29x1.40mm_HandSolder; Campo4 (none) -> ERA-6AEB6043V
- R20: value 1K -> 604K; footprint Resistor_SMD:R_0805_2012Metric_Pad1.15x1.50mm_HandSolder -> Resistor_SMD:R_0805_2012Metric_Pad1.29x1.40mm_HandSolder; Campo4 (none) -> ERA-6AEB6043V
- R21: value 43.5K -> 10k; footprint Resistor_SMD:R_0805_2012Metric_Pad1.15x1.50mm_HandSolder -> Resistor_SMD:R_0805_2012Metric_Pad1.29x1.40mm_HandSolder; Campo4 (none) -> RR1220P-103-D
- R4, R5: value 10K -> 2.2K; Campo4 (none) -> ERA-6AEB222V
- R6, R7: Campo4 (none) -> RR1220P-103-D
- U1: Campo4 (none) -> USBLC6-2SC6
- U11: Campo4 (none) -> TLA2024IRUGT
- U2: Campo4 (none) -> OM-O2P
Connections:
- net +3V3: no longer U1.5 (Vbus)
- net +5V: now also J1.1 (VBUS), U1.5 (Vbus), U12.8 (VCC)
- net GND: now also R21.2, BT1.2 (-), D5.2 (-), D6.1 (K), U12.4 (GND); no longer R20.2
- net SCL: now also U12.6 (SCL)
- net SDA: now also U2.17 (5/I2C_SDA), U12.5 (SDA)
- net V_TEST: now also R20.2, R21.1; no longer R19.2, R20.1
- net Vac: now also D5.3 (~~)
- net error: now reaches U2.2 (11)
- net error: now also R22.1
- net at R19.1: now also D5.1 (+); no longer R21.2
- new net: U12.1 (X1), Y1.1
- new net: U12.2 (X2), Y1.2
- new net: D6.2 (A), R22.2
- new net: R19.2, R20.1
- new net +BATT: BT1.1 (+), U12.3 (VBAT)
- new net Nac: D5.4 (~~)

Commit message: pasandome a mac
Parts:
- removed J1: USB_B_Micro, Devices_MSS:USB_Micro-B_10118193-0001LF, symbol Connector_Specialized:USB_B_Micro
- removed U1: USBLC6-2, Package_TO_SOT_SMD:SOT-23-6_Handsoldering, symbol omega-dock-new:USBLC6-2
- added D4, D7: LED, LED_SMD:LED_0603_1608Metric_Castellated, symbol Device:LED_ALT
- added J1: SI, Devices_MSS:HE_XDF1B_1x03_P2.50mm_Horizontal, symbol Connector_Generic:Conn_01x03
- added R23: 10K, Resistor_SMD:R_0805_2012Metric_Pad1.29x1.40mm_HandSolder, symbol Device:R
- added R24, R8: 100, Resistor_SMD:R_0805_2012Metric_Pad1.29x1.40mm_HandSolder, symbol Device:R
- added SW1: RST, Button_Switch_SMD:Panasonic_EVQPUL_EVQPUC, symbol Switch:SW_Push
- J2: value Conn_01x04 -> Termistor; Campo4 S4B-XH-A(LF)(SN) -> DF1BZ-4P-2.5DS
Connections:
- net labels added: +3V3, GPIO, VacF, red
- net labels removed: UD+, UD-, Vac
- wire segments 121 -> 127
- no-connect marks 20 -> 18
Other:
- note added: "address->0x48"
- moved on the sheet: D6, J2, R19, R20, R22, R4, R5, R6, R7
